Commit message: Update

File: robot_ws_ros2/install/nav2_simu/share/nav2_simu/src/description/bot_description.urdf (robot description, URDF)
Before this commit: robot bot, 4 links, 3 joints
Joints:
- removed joint footprint_joint
- added joint base_joint: type fixed, parent base_link, child base_footprint, origin xyz=0.0 0.0 ${-(wheels_radius+wheels_zoffset+square1_height/2)} rpy=0 0 0

File: robot_ws_ros2/src/nav2_simu/src/description/bot_description.urdf (robot description, URDF)
Before this commit: robot bot, 4 links, 3 joints
Joints:
- removed joint footprint_joint
- added joint base_joint: type fixed, parent base_link, child base_footprint, origin xyz=0.0 0.0 ${-(wheels_radius+wheels_zoffset+square1_height/2)} rpy=0 0 0

Commit message: Update

File: robot_ws_ros2/install/nav2_simu/share/nav2_simu/src/description/bot_description.urdf (robot description, URDF)
Before this commit: robot bot, 4 links, 3 joints
Links:
- added link base_sup_link; collision cylinder length=${wheels_radius*2} radius=${wheels_radius}; visual cylinder length=${wheels_radius+wheels_zoffset+0.1} radius=${wheels_radius}
- added link cam1_depth_frame
- added link cam1_link, mass 0.035; collision box size=0.015 0.130 0.022; visual box size=0.015 0.130 0.022
- added link cam2_depth_frame
- added link cam2_link, mass 0.035; collision box size=0.015 0.130 0.022; visual box size=0.015 0.130 0.022
- added link imu_link; collision box size=0.01 0.01 0.01; visual box size=0.01 0.01 0.01
- link base2_link: geometry collision box size=${square2_length} ${square2_length} ${square2_height*0.8}; visual box size=${square2_length} ${square2_length} ${square2_height}
Joints:
- added joint $base_sup_joint: type continuous, parent base_link, child base_sup_link, origin xyz=0.0 0.0 ${-((wheels_radius+wheels_zoffset+0.1)/2+(square1_height/2))} rpy=0 0 0, axis 0 0 1
- added joint cam1_depth_joint: type fixed, parent cam1_link, child cam1_depth_frame, origin xyz=0 0 0 rpy=${-pi/2} 0 ${-pi/2}
- added joint cam1_joint: type fixed, parent base3_link, child cam1_link, origin xyz=${(square1_length/2)+0.015/2} 0.0 ${(square2_height/2)-0.03-0.022/2} rpy=0.0 0.0 0.0
- added joint cam2_depth_joint: type fixed, parent cam2_link, child cam2_depth_frame, origin xyz=0 0 0 rpy=${-pi/2} 0 ${-pi/2}
- added joint cam2_joint: type fixed, parent base3_link, child cam2_link, origin xyz=${-((square1_length/2)+0.015/2)} 0.0 ${(square2_height/2)-0.03-0.022/2} rpy=0.0 0.0 ${pi}
- added joint imu_joint: type fixed, parent base_link, child imu_link, origin xyz=0 0 0.0
- joint base_joint: origin xyz=0.0 0.0 ${-(wheels_radius+wheels_zoffset+square1_height/2)} rpy=0 0 0 -> xyz=0.0 0.0 ${-(wheels_radius*2+wheels_zoffset+square1_height/2)} rpy=0 0 0

File: robot_ws_ros2/src/nav2_simu/src/description/bot_description.urdf (robot description, URDF)
Before this commit: robot bot, 4 links, 3 joints
Links:
- added link base_sup_link; collision cylinder length=${wheels_radius*2} radius=${wheels_radius}; visual cylinder length=${wheels_radius+wheels_zoffset+0.1} radius=${wheels_radius}
- added link cam1_depth_frame
- added link cam1_link, mass 0.035; collision box size=0.015 0.130 0.022; visual box size=0.015 0.130 0.022
- added link cam2_depth_frame
- added link cam2_link, mass 0.035; collision box size=0.015 0.130 0.022; visual box size=0.015 0.130 0.022
- added link imu_link; collision box size=0.01 0.01 0.01; visual box size=0.01 0.01 0.01
- link base2_link: geometry collision box size=${square2_length} ${square2_length} ${square2_height*0.8}; visual box size=${square2_length} ${square2_length} ${square2_height}
Joints:
- added joint $base_sup_joint: type continuous, parent base_link, child base_sup_link, origin xyz=0.0 0.0 ${-((wheels_radius+wheels_zoffset+0.1)/2+(square1_height/2))} rpy=0 0 0, axis 0 0 1
- added joint cam1_depth_joint: type fixed, parent cam1_link, child cam1_depth_frame, origin xyz=0 0 0 rpy=${-pi/2} 0 ${-pi/2}
- added joint cam1_joint: type fixed, parent base3_link, child cam1_link, origin xyz=${(square1_length/2)+0.015/2} 0.0 ${(square2_height/2)-0.03-0.022/2} rpy=0.0 0.0 0.0
- added joint cam2_depth_joint: type fixed, parent cam2_link, child cam2_depth_frame, origin xyz=0 0 0 rpy=${-pi/2} 0 ${-pi/2}
- added joint cam2_joint: type fixed, parent base3_link, child cam2_link, origin xyz=${-((square1_length/2)+0.015/2)} 0.0 ${(square2_height/2)-0.03-0.022/2} rpy=0.0 0.0 ${pi}
- added joint imu_joint: type fixed, parent base_link, child imu_link, origin xyz=0 0 0.0
- joint base_joint: origin xyz=0.0 0.0 ${-(wheels_radius+wheels_zoffset+square1_height/2)} rpy=0 0 0 -> xyz=0.0 0.0 ${-(wheels_radius*2+wheels_zoffset+square1_height/2)} rpy=0 0 0

Commit message: new world

File: robot_ws_ros2/install/nav2_simu/share/nav2_simu/src/description/bot_description.urdf (robot description, URDF)
Before this commit: robot bot, 10 links, 9 joints
Links:
- removed link base_sup_link
- removed link cam1_depth_frame
- removed link cam1_link
- removed link cam2_depth_frame
- removed link cam2_link
- added link camb_depth_frame
- added link camb_link, mass 0.035; collision box size=0.015 0.130 0.022; visual box size=0.015 0.130 0.022
- added link camf_depth_frame
- added link camf_link, mass 0.035; collision box size=0.015 0.130 0.022; visual box size=0.015 0.130 0.022
Joints:
- removed joint $base_sup_joint
- removed joint cam1_depth_joint
- removed joint cam1_joint
- removed joint cam2_depth_joint
- removed joint cam2_joint
- added joint camb_depth_joint: type fixed, parent camb_link, child camb_depth_frame, origin xyz=0 0 0 rpy=${-pi/2} 0 ${-pi/2}
- added joint camb_joint: type fixed, parent base3_link, child camb_link, origin xyz=${-((square1_length/2)+0.015/2)} 0.0 ${(square2_height/2)-0.03-0.022/2} rpy=0.0 0.0 ${pi}
- added joint camf_depth_joint: type fixed, parent camf_link, child camf_depth_frame, origin xyz=0 0 0 rpy=${-pi/2} 0 ${-pi/2}
- added joint camf_joint: type fixed, parent base3_link, child camf_link, origin xyz=${(square1_length/2)+0.015/2} 0.0 ${(square2_height/2)-0.03-0.022/2} rpy=0.0 0.0 0.0
