Commit message: Upates

File: robot_ws_ros2/src/call_m_supervisor/description/bot/camera_imu_description.urdf.xacro (robot description, xacro)
@@ -4,5 +4,5 @@
 	<!--2 CAMERA-->
 	<!--camera object front-->
-	<link name="camf_link">
+	<link name="cam1_link">
 		<visual>
 		<origin xyz="0 0 0" rpy="0 0 0"/>
@@ -23,23 +23,23 @@
 		</inertial>
 	</link>
-	<joint name="camf_joint" type="fixed">
+	<joint name="cam1_joint" type="fixed">
 		<parent link="base3_link"/>
-		<child link="camf_link"/>
-		<origin xyz="${(square1_length/2)+0.015/2} 0.0 ${(square2_height/2)-0.03-0.022/2}" rpy="0.0 0.0 0.0"/>
+		<child link="cam1_link"/>
+		<origin xyz="0.0 ${(square1_length/2)+0.015/2} ${(square3_height/2)-0.03-0.022/2}" rpy="0.0 0.0 ${pi/2}"/>
 	</joint>
 	<!--depth camera front-->
-	<link name="camf_depth_frame"/>
-	<joint name="camf_depth_joint" type="fixed">
+	<link name="cam1_depth_frame"/>
+	<joint name="cam1_depth_joint" type="fixed">
 		<origin xyz="0 0 0" rpy="${-pi/2} 0 ${-pi/2}"/>
-		<parent link="camf_link"/>
-		<child link="camf_depth_frame"/>
-	</joint>
-	<gazebo reference="camf_link">
+		<parent link="cam1_link"/>
+		<child link="cam1_depth_frame"/>
+	</joint>
+	<gazebo reference="cam1_link">
 		<!-- Gazebo is unable to use the same <material> tags that are already in the URDF (that RViz uses). -->
     	<!-- Instead, we need to add gazebo tags for our links that refer to Gazebo materials -->
         <material>Gazebo/Orange</material>
-		<sensor type="depth" name="camf">
+		<sensor type="depth" name="cam1">
 		<update_rate>30.0</update_rate>
-		<camera name="camf_cam">
+		<camera name="cam1_cam">
 			<horizontal_fov>1.6</horizontal_fov>
 			<image>
@@ -62,5 +62,5 @@
 			<alwaysOn>true</alwaysOn>
 			<updateRate>0.0</updateRate>
-			<frame_name>camf_depth_frame</frame_name>
+			<frame_name>cam1_depth_frame</frame_name>
 			<pointCloudCutoff>0.5</pointCloudCutoff>
 			<pointCloudCutoffMax>3.0</pointCloudCutoffMax>
@@ -79,5 +79,5 @@
 	</gazebo>
 	<!--camera object back-->
-	<link name="camb_link">
+	<link name="cam2_link">
 		<visual>
 		<origin xyz="0 0 0" rpy="0 0 0"/>
@@ -98,23 +98,23 @@
 		</inertial>
 	</link>
-	<joint name="camb_joint" type="fixed">
+	<joint name="cam2_joint" type="fixed">
 		<parent link="base3_link"/>
-		<child link="camb_link"/>
-		<origin xyz="${-((square1_length/2)+0.015/2)} 0.0 ${(square2_height/2)-0.03-0.022/2}" rpy="0.0 0.0 ${pi}"/>
+		<child link="cam2_link"/>
+		<origin xyz="0.0 ${-((square1_length/2)+0.015/2)} ${(square3_height/2)-0.03-0.022/2}" rpy="0.0 0.0 ${-pi/2}"/>
 	</joint>
 	<!--depth camera back-->
-	<link name="camb_depth_frame"/>
-	<joint name="camb_depth_joint" type="fixed">
+	<link name="cam2_depth_frame"/>
+	<joint name="cam2_depth_joint" type="fixed">
 		<origin xyz="0 0 0" rpy="${-pi/2} 0 ${-pi/2}"/>
-		<parent link="camb_link"/>
-		<child link="camb_depth_frame"/>
-	</joint>
-	<gazebo reference="camb_link">
+		<parent link="cam2_link"/>
+		<child link="cam2_depth_frame"/>
+	</joint>
+	<gazebo reference="cam2_link">
 		<!-- Gazebo is unable to use the same <material> tags that are already in the URDF (that RViz uses). -->
     	<!-- Instead, we need to add gazebo tags for our links that refer to Gazebo materials -->
         <material>Gazebo/Orange</material>
-		<sensor type="depth" name="camb">
+		<sensor type="depth" name="cam2">
 		<update_rate>30.0</update_rate>
-		<camera name="camb_cam">
+		<camera name="cam2_cam">
 			<horizontal_fov>1.6</horizontal_fov>
 			<image>
@@ -137,5 +137,5 @@
 			<alwaysOn>true</alwaysOn>
 			<updateRate>0.0</updateRate>
-			<frame_name>camb_depth_frame</frame_name>
+			<frame_name>cam2_depth_frame</frame_name>
 			<pointCloudCutoff>0.5</pointCloudCutoff>
 			<pointCloudCutoffMax>3.0</pointCloudCutoffMax>

File: robot_ws_ros2/src/call_m_supervisor/description/bot/lidars_description.urdf.xacro (robot description, xacro)
@@ -3,5 +3,5 @@
 	<!-- THIS FILE NEED TO BE INCLUDED IN 'bot_description.urdf.xacro' -->
 	<!--2 LIDAR-->
-	<xacro:macro name="lidar" params="prefix x y">
+	<xacro:macro name="lidar" params="prefix x y alpha">
 		<link name="${prefix}_link">
 			<inertial>
@@ -26,5 +26,5 @@
 			<parent link="base_link"/>
 			<child link="${prefix}_link"/>
-			<origin xyz="${x} ${y} ${square1_height/2+0.1/2}" rpy="0 0 0"/>
+			<origin xyz="${x} ${y} ${square1_height/2+0.1/2}" rpy="0 0 ${alpha}"/>
 		</joint>
 		<gazebo reference="${prefix}_link">
@@ -67,5 +67,5 @@
 		</gazebo>
 	</xacro:macro>
-	<xacro:lidar prefix="lidar1" x="${(square1_length/2)-0.0508}" y="${(square1_length/2)-0.0508}" />
-	<xacro:lidar prefix="lidar2" x="${-((square1_length/2)-0.0508)}" y="${-((square1_length/2)-0.0508)}" />
+	<xacro:lidar prefix="lidar1" x="${(square1_length/2)-0.0508}" y="${(square1_length/2)-0.0508}" alpha="${-3*pi/4}" />
+	<xacro:lidar prefix="lidar2" x="${-((square1_length/2)-0.0508)}" y="${-((square1_length/2)-0.0508)}" alpha="${pi/4}" />
 </robot>

Commit message: Update

File: robot_ws_ros2/src/call_m_supervisor/description/bot/camera_imu_description.urdf.xacro (robot description, xacro)
@@ -23,8 +23,9 @@
 		</inertial>
 	</link>
-	<joint name="cam1_joint" type="fixed">
+	<joint name="cam1_joint" type="continuous">
 		<parent link="base3_link"/>
 		<child link="cam1_link"/>
 		<origin xyz="${(square1_length/2)+0.015/2} 0.0 ${(square3_height/2)-0.03-0.022/2}" rpy="0.0 0.0 0.0"/>
+		<axis xyz="0 1 0"/>
 	</joint>
 	<!--depth camera front-->
@@ -40,5 +41,5 @@
         <material>Gazebo/Orange</material>
 		<sensor type="depth" name="cam1">
-		<update_rate>30.0</update_rate>
+		<update_rate>100</update_rate>
 		<camera name="cam1_cam">
 			<horizontal_fov>1.6</horizontal_fov>
@@ -107,8 +108,9 @@
 		</inertial>
 	</link>
-	<joint name="cam2_joint" type="fixed">
+	<joint name="cam2_joint" type="continuous">
 		<parent link="base3_link"/>
 		<child link="cam2_link"/>
 		<origin xyz="${-((square1_length/2)+0.015/2)} 0.0 ${(square3_height/2)-0.03-0.022/2}" rpy="0.0 0.0 ${pi}"/>
+		<axis xyz="0 1 0"/>
 	</joint>
 	<!--depth camera back-->
@@ -124,5 +126,5 @@
         <material>Gazebo/Orange</material>
 		<sensor type="depth" name="cam2">
-		<update_rate>30.0</update_rate>
+		<update_rate>100</update_rate>
 		<camera name="cam2_cam">
 			<horizontal_fov>1.6</horizontal_fov>

File: robot_ws_ros2/src/call_m_supervisor/description/bot/gazebo_template.urdf.xacro (robot description, xacro)
@@ -7,5 +7,5 @@
         <plugin name="gazebo_ros_joint_state_publisher"
             filename="libgazebo_ros_joint_state_publisher.so">
-            <update_rate>20</update_rate>
+            <update_rate>100</update_rate>
             <joint_name>wheel_2_sup_joint</joint_name>
             <joint_name>wheel_3_sup_joint</joint_name>
@@ -14,4 +14,6 @@
             <joint_name>wheel_3_joint</joint_name>
             <joint_name>wheel_1_joint</joint_name>
+            <joint_name>cam1_joint</joint_name>
+            <joint_name>cam2_joint</joint_name>
         </plugin>
     </gazebo>

File: robot_ws_ros2/src/call_m_supervisor/description/bot/lidars_description.urdf.xacro (robot description, xacro)
@@ -36,5 +36,5 @@
 			<always_on>true</always_on>
 			<visualize>true</visualize>
-			<update_rate>5</update_rate>
+			<update_rate>100</update_rate>
 			<ray>
 				<scan>

File: robot_ws_ros2/src/call_m_supervisor/description/bot/ros2_control.xacro (robot description, xacro)
@@ -42,4 +42,16 @@
             </command_interface>
         </joint>
+        <joint name="cam1_joint">
+            <command_interface name="position">
+                <param name="min">-100</param>
+                <param name="max">100</param>
+            </command_interface>
+        </joint>
+        <joint name="cam2_joint">
+            <command_interface name="position">
+                <param name="min">-100</param>
+                <param name="max">100</param>
+            </command_interface>
+        </joint>
     </ros2_control>
     <!--we set up gazebo tag to indicate that we use ros2 control, a controller manager is integrated in it, so we need to indicate wich controller to use in yaml file-->
