Commit message: Update

File: robot_ws_ros2/src/call_m_supervisor/description/bot/cameras_description.urdf.xacro (robot description, xacro)
@@ -18,5 +18,5 @@
 		<xacro:property name="optical_offset_x" value="0.0" />
 		<!-- Camera mounting point (the threaded screw hole in the bottom) -->
-		<link name="${name}_link">
+		<link name="${name}_camera_link">
 			<visual>
 			<origin xyz="0 0 0" rpy="0 0 0"/>
@@ -33,5 +33,5 @@
 		<joint name="${name}_joint" type="continuous">
 			<parent link="base3_link"/>
-			<child link="${name}_link"/>
+			<child link="${name}_camera_link"/>
 			<origin xyz="${x} ${y} ${z}" rpy="0.0 0.0 ${rot_z}"/>
 			<axis xyz="0 1 0"/>
@@ -55,5 +55,5 @@
 		</link>
 		<joint name="${name}_camera_center_joint" type="fixed">
-		<parent link="${name}_link"/>
+		<parent link="${name}_camera_link"/>
 		<child link="${name}_camera_center"/>
 		<origin xyz="0 0 0" rpy="0 ${bottom_slope} 0" />
@@ -93,8 +93,8 @@
 	<joint name="cam1_depth_joint" type="fixed">
 		<origin xyz="0 0 0" rpy="${-pi/2} 0 ${-pi/2}"/>
-		<parent link="cam1_link"/>
+		<parent link="cam1_camera_link"/>
 		<child link="cam1_depth_frame"/>
 	</joint>
-	<gazebo reference="cam1_link">
+	<gazebo reference="cam1_camera_link">
 		<!-- Gazebo is unable to use the same <material> tags that are already in the URDF (that RViz uses). -->
     	<!-- Instead, we need to add gazebo tags for our links that refer to Gazebo materials -->
@@ -152,8 +152,8 @@
 	<joint name="cam2_depth_joint" type="fixed">
 		<origin xyz="0 0 0" rpy="${-pi/2} 0 ${-pi/2}"/>
-		<parent link="cam2_link"/>
+		<parent link="cam2_camera_link"/>
 		<child link="cam2_depth_frame"/>
 	</joint>
-	<gazebo reference="cam2_link">
+	<gazebo reference="cam2_camera_link">
 		<!-- Gazebo is unable to use the same <material> tags that are already in the URDF (that RViz uses). -->
     	<!-- Instead, we need to add gazebo tags for our links that refer to Gazebo materials -->
