Commit message: Update

File: robot_ws_ros2/src/call_m_supervisor/description/bot/bot_description.urdf.xacro (robot description, xacro)
@@ -101,4 +101,27 @@
 		<origin xyz="0.0 0.0 ${(square1_height/2)+square2_height+(square3_height/2)}" rpy="0 0 0"/>
 	</joint>
+	<!-- Robot Support, to be deleted want controlling (TBM)-->
+	<link name="base_sup_link">
+		<visual>
+		<geometry>
+			<cylinder radius="${wheels_radius}" length="${wheels_radius+wheels_zoffset+0.1}"/>
+		</geometry>
+		<material name="Cyan">
+			<color rgba="0 1.0 1.0 1.0"/>
+		</material>
+		</visual>
+		<collision>
+		<origin xyz="0 0 0" rpy="0 0 0"/>
+		<geometry>
+			<cylinder radius="${wheels_radius}" length="${wheels_radius*2}"/>
+		</geometry>
+		</collision>
+		<xacro:cylinder_inertia m="20" r="${wheels_radius}" h="${wheels_radius+wheels_zoffset+0.1}"/>
+	</link>
+	<joint name="$base_sup_joint" type="fixed">
+		<parent link="base_link"/>
+		<child link="base_sup_link"/>
+		<origin xyz="0.0 0.0 ${-((wheels_radius+wheels_zoffset+0.1)/2+(square1_height/2))}" rpy="0 0 0"/>
+	</joint>
 	<!-- Robot Footprint-->
 	<link name="base_footprint">
@@ -171,7 +194,7 @@
 		</joint>
 	</xacro:macro>
-	<xacro:wheel prefix="wheel_f" angle="0.0" type="sphere" />
-	<xacro:wheel prefix="wheel_bl" angle="${2*pi/3}" type="sphere" />
-	<xacro:wheel prefix="wheel_br" angle="${-2*pi/3}" type="sphere" />
+	<xacro:wheel prefix="wheel_2" angle="${-pi/2}" type="sphere" />
+	<xacro:wheel prefix="wheel_3" angle="${(2*pi/3)-pi/2}" type="sphere" />
+	<xacro:wheel prefix="wheel_1" angle="${(-2*pi/3)-pi/2}" type="sphere" />
 	<!--Gazebo plugin to read all transmission tags-->
 	<!--

File: robot_ws_ros2/src/call_m_supervisor/description/bot/camera_imu_description.urdf.xacro (robot description, xacro)
@@ -26,5 +26,5 @@
 		<parent link="base3_link"/>
 		<child link="cam1_link"/>
-		<origin xyz="0.0 ${(square1_length/2)+0.015/2} ${(square3_height/2)-0.03-0.022/2}" rpy="0.0 0.0 ${pi/2}"/>
+		<origin xyz="${(square1_length/2)+0.015/2} 0.0 ${(square3_height/2)-0.03-0.022/2}" rpy="0.0 0.0 0.0"/>
 	</joint>
 	<!--depth camera front-->
@@ -59,4 +59,13 @@
 		</camera>
 		<plugin name="depth_camera_controller" filename="libgazebo_ros_camera.so">
+			<!--/cam1/zed_node/rgb/image_rect_color-->
+		    <ros>
+                <namespace>cam1</namespace>
+                <remapping>cam1/image_raw:=zed_node/rgb/image_rect_color</remapping>
+                <remapping>cam1/depth/image_raw:=depth/image_rect_raw</remapping>
+                <remapping>cam1/camera_info:=camera_info</remapping>
+                <remapping>cam1/depth/camera_info:=depth/camera_info</remapping>
+                <remapping>cam1/points:=depth/points</remapping>
+            </ros>
 			<baseline>0.2</baseline>
 			<alwaysOn>true</alwaysOn>
@@ -101,5 +110,5 @@
 		<parent link="base3_link"/>
 		<child link="cam2_link"/>
-		<origin xyz="0.0 ${-((square1_length/2)+0.015/2)} ${(square3_height/2)-0.03-0.022/2}" rpy="0.0 0.0 ${-pi/2}"/>
+		<origin xyz="${-((square1_length/2)+0.015/2)} 0.0 ${(square3_height/2)-0.03-0.022/2}" rpy="0.0 0.0 ${pi}"/>
 	</joint>
 	<!--depth camera back-->
@@ -134,4 +143,12 @@
 		</camera>
 		<plugin name="depth_camera_controller" filename="libgazebo_ros_camera.so">
+			<ros>
+                <namespace>cam2</namespace>
+                <remapping>cam2/image_raw:=zed_node/rgb/image_rect_color</remapping>
+                <remapping>cam2/depth/image_raw:=depth/image_rect_raw</remapping>
+                <remapping>cam2/camera_info:=camera_info</remapping>
+                <remapping>cam2/depth/camera_info:=depth/camera_info</remapping>
+                <remapping>cam2/points:=depth/points</remapping>
+            </ros>
 			<baseline>0.2</baseline>
 			<alwaysOn>true</alwaysOn>

File: robot_ws_ros2/src/call_m_supervisor/description/bot/gazebo_template.urdf.xacro (robot description, xacro)
@@ -8,10 +8,10 @@
             filename="libgazebo_ros_joint_state_publisher.so">
             <update_rate>20</update_rate>
-            <joint_name>wheel_f_sup_joint</joint_name>
-            <joint_name>wheel_bl_sup_joint</joint_name>
-            <joint_name>wheel_br_sup_joint</joint_name>
-            <joint_name>wheel_f_joint</joint_name>
-            <joint_name>wheel_bl_joint</joint_name>
-            <joint_name>wheel_br_joint</joint_name>
+            <joint_name>wheel_2_sup_joint</joint_name>
+            <joint_name>wheel_3_sup_joint</joint_name>
+            <joint_name>wheel_1_sup_joint</joint_name>
+            <joint_name>wheel_2_joint</joint_name>
+            <joint_name>wheel_3_joint</joint_name>
+            <joint_name>wheel_1_joint</joint_name>
         </plugin>
     </gazebo>
@@ -21,5 +21,5 @@
             e.g. <dynamics damping="10.0" friction="10.0"/> -->
     <!-- Here's an example message to publish to test it:
-    ros2 topic pub -1 /set_joint_trajectory trajectory_msgs/msg/JointTrajectory  '{header: {frame_id: base_link}, joint_names: [wheel_f_sup_joint,wheel_bl_sup_joint,wheel_br_sup_joint,wheel_f_joint,wheel_bl_joint,wheel_br_joint], points: [  {positions: {0.8,0.6,0.8,0.6,0.8,0.6}} ]}'
+    ros2 topic pub -1 /set_joint_trajectory trajectory_msgs/msg/JointTrajectory  '{header: {frame_id: base_link}, joint_names: [wheel_2_sup_joint,wheel_3_sup_joint,wheel_1_sup_joint,wheel_2_joint,wheel_3_joint,wheel_1_joint], points: [  {positions: {0.8,0.6,0.8,0.6,0.8,0.6}} ]}'
      -->
     <gazebo>

File: robot_ws_ros2/src/call_m_supervisor/description/bot/lidars_description.urdf.xacro (robot description, xacro)
@@ -42,11 +42,11 @@
 					<samples>360</samples>
 					<resolution>1.000000</resolution>
-					<min_angle>0.000000</min_angle>
-					<max_angle>6.280000</max_angle>
+					<min_angle>3.14159265359</min_angle> <!-- Set to π for 180 degrees (We need to shift all values according to rpLidars)-->
+					<max_angle>${6.28318530718+3.14159265359}</max_angle> <!-- Set to 3π for keeping 360 degres range -->
 				</horizontal>
 				</scan>
 				<range>
-				<min>0.120000</min>
-				<max>3.5</max>
+				<min>0.07</min>
+				<max>12.0</max>
 				<resolution>0.015000</resolution>
 				</range>
@@ -67,5 +67,5 @@
 		</gazebo>
 	</xacro:macro>
-	<xacro:lidar prefix="lidar1" x="${(square1_length/2)-0.0508}" y="${(square1_length/2)-0.0508}" alpha="${-3*pi/4}" />
-	<xacro:lidar prefix="lidar2" x="${-((square1_length/2)-0.0508)}" y="${-((square1_length/2)-0.0508)}" alpha="${pi/4}" />
+	<xacro:lidar prefix="lidar1" x="${(square1_length/2)-0.0508}" y="${-((square1_length/2)-0.0508)}" alpha="${3*pi/4}" />
+	<xacro:lidar prefix="lidar2" x="${-((square1_length/2)-0.0508)}" y="${(square1_length/2)-0.0508}" alpha="${-pi/4}" />
 </robot>

Commit message: Update

File: robot_ws_ros2/src/call_m_supervisor/description/bot/bot_description.urdf.xacro (robot description, xacro)
@@ -197,15 +197,8 @@
 	<xacro:wheel prefix="wheel_3" angle="${(2*pi/3)-pi/2}" type="sphere" />
 	<xacro:wheel prefix="wheel_1" angle="${(-2*pi/3)-pi/2}" type="sphere" />
-	<!--Gazebo plugin to read all transmission tags-->
-	<!--
-	<gazebo>
-	<plugin name="gazebo_ros_control" filename="libgazebo_ros2_control.so">
-		<robotNamespace>/simubot</robotNamespace>
-	</plugin>
-	</gazebo>
-	-->
 	<xacro:include filename="lidars_description.urdf.xacro"/>
 	<xacro:include filename="camera_imu_description.urdf.xacro"/>
 	<xacro:include filename="gazebo_template.urdf.xacro"/>
+	<xacro:include filename="ros2_control.xacro"/>
 	<!--Keep this at the end, Used as debug, whrn changing the color we can know if the model loaded by gazebo is really this one
 	or a previous working version.if the color of base2_link match the color specified on Gazebo, then everything worked correctly-->

File: robot_ws_ros2/src/call_m_supervisor/description/bot/gazebo_template.urdf.xacro (robot description, xacro)
@@ -16,16 +16,3 @@
         </plugin>
     </gazebo>
-    <!-- This plugin will read a JointTrajectory message from the /set_joint_trajectory topic
-            and move the machine accordingly. It's a bit clunky but it works. -->
-    <!-- You'll probably want to add damping to the joints to stop them it flopping around.
-            e.g. <dynamics damping="10.0" friction="10.0"/> -->
-    <!-- Here's an example message to publish to test it:
-    ros2 topic pub -1 /set_joint_trajectory trajectory_msgs/msg/JointTrajectory  '{header: {frame_id: base_link}, joint_names: [wheel_2_sup_joint,wheel_3_sup_joint,wheel_1_sup_joint,wheel_2_joint,wheel_3_joint,wheel_1_joint], points: [  {positions: {0.8,0.6,0.8,0.6,0.8,0.6}} ]}'
-     -->
-    <gazebo>
-        <plugin name="gazebo_ros_joint_pose_trajectory"
-            filename="libgazebo_ros_joint_pose_trajectory.so">
-            <update_rate>2</update_rate>
-        </plugin>
-    </gazebo>
 </robot>

Commit message: Update

File: robot_ws_ros2/src/call_m_supervisor/description/bot/bot_description.urdf.xacro (robot description, xacro)
@@ -101,27 +101,4 @@
 		<origin xyz="0.0 0.0 ${(square1_height/2)+square2_height+(square3_height/2)}" rpy="0 0 0"/>
 	</joint>
-	<!-- Robot Support, to be deleted want controlling (TBM)-->
-	<link name="base_sup_link">
-		<visual>
-		<geometry>
-			<cylinder radius="${wheels_radius}" length="${wheels_radius+wheels_zoffset+0.1}"/>
-		</geometry>
-		<material name="Cyan">
-			<color rgba="0 1.0 1.0 1.0"/>
-		</material>
-		</visual>
-		<collision>
-		<origin xyz="0 0 0" rpy="0 0 0"/>
-		<geometry>
-			<cylinder radius="${wheels_radius}" length="${wheels_radius*2}"/>
-		</geometry>
-		</collision>
-		<xacro:cylinder_inertia m="20" r="${wheels_radius}" h="${wheels_radius+wheels_zoffset+0.1}"/>
-	</link>
-	<joint name="$base_sup_joint" type="fixed">
-		<parent link="base_link"/>
-		<child link="base_sup_link"/>
-		<origin xyz="0.0 0.0 ${-((wheels_radius+wheels_zoffset+0.1)/2+(square1_height/2))}" rpy="0 0 0"/>
-	</joint>
 	<!-- Robot Footprint-->
 	<link name="base_footprint">

File: robot_ws_ros2/src/call_m_supervisor/description/bot/ros2_control.xacro (robot description, xacro)
@@ -12,4 +12,34 @@
             </command_interface>
         </joint>
+        <joint name="wheel_2_joint">
+            <command_interface name="velocity">
+                <param name="min">-100</param>
+                <param name="max">100</param>
+            </command_interface>
+        </joint>
+        <joint name="wheel_3_joint">
+            <command_interface name="velocity">
+                <param name="min">-100</param>
+                <param name="max">100</param>
+            </command_interface>
+        </joint>
+        <joint name="wheel_1_sup_joint">
+            <command_interface name="position">
+                <param name="min">-100</param>
+                <param name="max">100</param>
+            </command_interface>
+        </joint>
+        <joint name="wheel_2_sup_joint">
+            <command_interface name="position">
+                <param name="min">-100</param>
+                <param name="max">100</param>
+            </command_interface>
+        </joint>
+        <joint name="wheel_3_sup_joint">
+            <command_interface name="position">
+                <param name="min">-100</param>
+                <param name="max">100</param>
+            </command_interface>
+        </joint>
     </ros2_control>
     <!--we set up gazebo tag to indicate that we use ros2 control, a controller manager is integrated in it, so we need to indicate wich controller to use in yaml file-->

Commit message: Update

File: robot_ws_ros2/src/call_m_supervisor/description/bot/bot_description.urdf.xacro (robot description, xacro)
@@ -101,4 +101,19 @@
 		<origin xyz="0.0 0.0 ${(square1_height/2)+square2_height+(square3_height/2)}" rpy="0 0 0"/>
 	</joint>
+	<link name="base4_link">
+		<visual>
+		<geometry>
+			<box size="${square1_length/4} ${square1_length/30} ${0.04}"/>
+		</geometry>
+		<material name="Green">
+			<color rgba="1.0 0.0 1.0 1.0"/>
+		</material>
+		</visual>
+	</link>
+	<joint name="base4_joint" type="fixed">
+		<parent link="base3_link"/>
+		<child link="base4_link"/>
+		<origin xyz="${square1_length/2-square1_length/4} 0.0 ${(square3_height/2)+0.02}" rpy="0 0 0"/>
+	</joint>
 	<!-- Robot Footprint-->
 	<link name="base_footprint">
@@ -178,4 +193,7 @@
 	<xacro:include filename="gazebo_template.urdf.xacro"/>
 	<xacro:include filename="ros2_control.xacro"/>
+	<gazebo reference="base4_link">
+		<material>Gazebo/Purple</material>
+	</gazebo>
 	<!--Keep this at the end, Used as debug, whrn changing the color we can know if the model loaded by gazebo is really this one
 	or a previous working version.if the color of base2_link match the color specified on Gazebo, then everything worked correctly-->

File: robot_ws_ros2/src/call_m_supervisor/description/bot/camera_imu_description.urdf.xacro (robot description, xacro)
@@ -2,6 +2,10 @@
 <robot name="bot" xmlns:xacro="http://ros.org/wiki/xacro">
 	<!-- THIS FILE NEED TO BE INCLUDED IN 'bot_description.urdf.xacro' -->
-	<!--2 CAMERA-->
-	<!--camera object front-->
+	<!--
+		////////////////////////
+		//////2 CAMERAS////////
+		///////////////////////
+	-->
+	<!--CAMERA 1 : FRONT-->
 	<link name="cam1_link">
 		<visual>
@@ -29,5 +33,5 @@
 		<axis xyz="0 1 0"/>
 	</joint>
-	<!--depth camera front-->
+	<!--depth sensor-->
 	<link name="cam1_depth_frame"/>
 	<joint name="cam1_depth_joint" type="fixed">
@@ -88,5 +92,92 @@
 		</sensor>
 	</gazebo>
-	<!--camera object back-->
+	<!--imu sensor-->
+	<link name="imu1_link">
+		<visual>
+		<geometry>
+			<box size="0.01 0.01 0.01"/>
+		</geometry>
+		</visual>
+		<collision>
+		<geometry>
+			<box size="0.01 0.01 0.01"/>
+		</geometry>
+		</collision>
+		<xacro:box_inertia m="0.01" w="0.01" d="0.01" h="0.01"/>
+	</link>
+	<joint name="imu1_joint" type="fixed">
+		<parent link="cam1_link"/>
+		<child link="imu1_link"/>
+		<origin xyz="0 0 0.0"/>
+	</joint>
+	<gazebo reference="imu_link">
+		<sensor name="imu_sensor" type="imu">
+		<plugin filename="libgazebo_ros_imu_sensor.so" name="imu_plugin">
+			<ros>
+			<namespace>/imu</namespace>
+			<remapping>~/out:=data</remapping>
+			</ros>
+			<initial_orientation_as_reference>false</initial_orientation_as_reference>
+		</plugin>
+		<always_on>true</always_on>
+		<update_rate>100</update_rate>
+		<visualize>true</visualize>
+		<imu>
+			<angular_velocity>
+			<x>
+				<noise type="gaussian">
+				<mean>0.0</mean>
+				<stddev>2e-4</stddev>
+				<bias_mean>0.0000075</bias_mean>
+				<bias_stddev>0.0000008</bias_stddev>
+				</noise>
+			</x>
+			<y>
+				<noise type="gaussian">
+				<mean>0.0</mean>
+				<stddev>2e-4</stddev>
+				<bias_mean>0.0000075</bias_mean>
+				<bias_stddev>0.0000008</bias_stddev>
+				</noise>
+			</y>
+			<z>
+				<noise type="gaussian">
+				<mean>0.0</mean>
+				<stddev>2e-4</stddev>
+				<bias_mean>0.0000075</bias_mean>
+				<bias_stddev>0.0000008</bias_stddev>
+				</noise>
+			</z>
+			</angular_velocity>
+			<linear_acceleration>
+			<x>
+				<noise type="gaussian">
+				<mean>0.0</mean>
+				<stddev>1.7e-2</stddev>
+				<bias_mean>0.1</bias_mean>
+				<bias_stddev>0.001</bias_stddev>
+				</noise>
+			</x>
+			<y>
+				<noise type="gaussian">
+				<mean>0.0</mean>
+				<stddev>1.7e-2</stddev>
+				<bias_mean>0.1</bias_mean>
+				<bias_stddev>0.001</bias_stddev>
+				</noise>
+			</y>
+			<z>
+				<noise type="gaussian">
+				<mean>0.0</mean>
+				<stddev>1.7e-2</stddev>
+				<bias_mean>0.1</bias_mean>
+				<bias_stddev>0.001</bias_stddev>
+				</noise>
+			</z>
+			</linear_acceleration>
+		</imu>
+		</sensor>
+	</gazebo>
+	<!--CAMERA 2 : BACK-->
 	<link name="cam2_link">
 		<visual>
@@ -114,5 +205,5 @@
 		<axis xyz="0 1 0"/>
 	</joint>
-	<!--depth camera back-->
+	<!--depth sensor-->
 	<link name="cam2_depth_frame"/>
 	<joint name="cam2_depth_joint" type="fixed">

Commit message: Update

File: robot_ws_ros2/src/call_m_supervisor/description/bot/bot_description.urdf.xacro (robot description, xacro)
@@ -190,5 +190,6 @@
 	<xacro:wheel prefix="wheel_1" angle="${(-2*pi/3)-pi/2}" type="sphere" />
 	<xacro:include filename="lidars_description.urdf.xacro"/>
-	<xacro:include filename="camera_imu_description.urdf.xacro"/>
+	<xacro:include filename="cameras_description.urdf.xacro"/>
+	<xacro:include filename="imu_description.urdf.xacro"/>
 	<xacro:include filename="gazebo_template.urdf.xacro"/>
 	<xacro:include filename="ros2_control.xacro"/>

File: robot_ws_ros2/src/call_m_supervisor/description/bot/cameras_description.urdf.xacro (robot description, xacro)
@@ -92,91 +92,4 @@
 		</sensor>
 	</gazebo>
-	<!--imu sensor-->
-	<link name="imu1_link">
-		<visual>
-		<geometry>
-			<box size="0.01 0.01 0.01"/>
-		</geometry>
-		</visual>
-		<collision>
-		<geometry>
-			<box size="0.01 0.01 0.01"/>
-		</geometry>
-		</collision>
-		<xacro:box_inertia m="0.01" w="0.01" d="0.01" h="0.01"/>
-	</link>
-	<joint name="imu1_joint" type="fixed">
-		<parent link="cam1_link"/>
-		<child link="imu1_link"/>
-		<origin xyz="0 0 0.0"/>
-	</joint>
-	<gazebo reference="imu_link">
-		<sensor name="imu_sensor" type="imu">
-		<plugin filename="libgazebo_ros_imu_sensor.so" name="imu_plugin">
-			<ros>
-			<namespace>/imu</namespace>
-			<remapping>~/out:=data</remapping>
-			</ros>
-			<initial_orientation_as_reference>false</initial_orientation_as_reference>
-		</plugin>
-		<always_on>true</always_on>
-		<update_rate>100</update_rate>
-		<visualize>true</visualize>
-		<imu>
-			<angular_velocity>
-			<x>
-				<noise type="gaussian">
-				<mean>0.0</mean>
-				<stddev>2e-4</stddev>
-				<bias_mean>0.0000075</bias_mean>
-				<bias_stddev>0.0000008</bias_stddev>
-				</noise>
-			</x>
-			<y>
-				<noise type="gaussian">
-				<mean>0.0</mean>
-				<stddev>2e-4</stddev>
-				<bias_mean>0.0000075</bias_mean>
-				<bias_stddev>0.0000008</bias_stddev>
-				</noise>
-			</y>
-			<z>
-				<noise type="gaussian">
-				<mean>0.0</mean>
-				<stddev>2e-4</stddev>
-				<bias_mean>0.0000075</bias_mean>
-				<bias_stddev>0.0000008</bias_stddev>
-				</noise>
-			</z>
-			</angular_velocity>
-			<linear_acceleration>
-			<x>
-				<noise type="gaussian">
-				<mean>0.0</mean>
-				<stddev>1.7e-2</stddev>
-				<bias_mean>0.1</bias_mean>
-				<bias_stddev>0.001</bias_stddev>
-				</noise>
-			</x>
-			<y>
-				<noise type="gaussian">
-				<mean>0.0</mean>
-				<stddev>1.7e-2</stddev>
-				<bias_mean>0.1</bias_mean>
-				<bias_stddev>0.001</bias_stddev>
-				</noise>
-			</y>
-			<z>
-				<noise type="gaussian">
-				<mean>0.0</mean>
-				<stddev>1.7e-2</stddev>
-				<bias_mean>0.1</bias_mean>
-				<bias_stddev>0.001</bias_stddev>
-				</noise>
-			</z>
-			</linear_acceleration>
-		</imu>
-		</sensor>
-	</gazebo>
 	<!--CAMERA 2 : BACK-->
 	<link name="cam2_link">
@@ -263,90 +176,3 @@
 		</sensor>
 	</gazebo>
-	<!--2 IMU in each camera-->
-	<link name="imu_link">
-		<visual>
-		<geometry>
-			<box size="0.01 0.01 0.01"/>
-		</geometry>
-		</visual>
-		<collision>
-		<geometry>
-			<box size="0.01 0.01 0.01"/>
-		</geometry>
-		</collision>
-		<xacro:box_inertia m="0.01" w="0.01" d="0.01" h="0.01"/>
-	</link>
-	<joint name="imu_joint" type="fixed">
-		<parent link="base_link"/>
-		<child link="imu_link"/>
-		<origin xyz="0 0 0.0"/>
-	</joint>
-	<gazebo reference="imu_link">
-		<sensor name="imu_sensor" type="imu">
-		<plugin filename="libgazebo_ros_imu_sensor.so" name="imu_plugin">
-			<ros>
-			<namespace>/imu</namespace>
-			<remapping>~/out:=data</remapping>
-			</ros>
-			<initial_orientation_as_reference>false</initial_orientation_as_reference>
-		</plugin>
-		<always_on>true</always_on>
-		<update_rate>100</update_rate>
-		<visualize>true</visualize>
-		<imu>
-			<angular_velocity>
-			<x>
-				<noise type="gaussian">
-				<mean>0.0</mean>
-				<stddev>2e-4</stddev>
-				<bias_mean>0.0000075</bias_mean>
-				<bias_stddev>0.0000008</bias_stddev>
-				</noise>
-			</x>
-			<y>
-				<noise type="gaussian">
-				<mean>0.0</mean>
-				<stddev>2e-4</stddev>
-				<bias_mean>0.0000075</bias_mean>
-				<bias_stddev>0.0000008</bias_stddev>
-				</noise>
-			</y>
-			<z>
-				<noise type="gaussian">
-				<mean>0.0</mean>
-				<stddev>2e-4</stddev>
-				<bias_mean>0.0000075</bias_mean>
-				<bias_stddev>0.0000008</bias_stddev>
-				</noise>
-			</z>
-			</angular_velocity>
-			<linear_acceleration>
-			<x>
-				<noise type="gaussian">
-				<mean>0.0</mean>
-				<stddev>1.7e-2</stddev>
-				<bias_mean>0.1</bias_mean>
-				<bias_stddev>0.001</bias_stddev>
-				</noise>
-			</x>
-			<y>
-				<noise type="gaussian">
-				<mean>0.0</mean>
-				<stddev>1.7e-2</stddev>
-				<bias_mean>0.1</bias_mean>
-				<bias_stddev>0.001</bias_stddev>
-				</noise>
-			</y>
-			<z>
-				<noise type="gaussian">
-				<mean>0.0</mean>
-				<stddev>1.7e-2</stddev>
-				<bias_mean>0.1</bias_mean>
-				<bias_stddev>0.001</bias_stddev>
-				</noise>
-			</z>
-			</linear_acceleration>
-		</imu>
-		</sensor>
-	</gazebo>
 </robot>
