Commit message: Update

File: robot_ws_ros2/src/call_m_supervisor/description/bot/bot_description.urdf.xacro (robot description, xacro)
@@ -191,5 +191,5 @@
 	<xacro:include filename="lidars_description.urdf.xacro"/>
 	<xacro:include filename="cameras_description.urdf.xacro"/>
-	<!--The simulated IMU seems to be noisy too much even with no noise set, so we don't use it-->
+	<!--The simulated IMU seems to be noisy too much even with no noise set, so we don't use it for linear movement-->
 	<xacro:include filename="imu_description.urdf.xacro"/>
 	<xacro:include filename="gazebo_template.urdf.xacro"/>

File: robot_ws_ros2/src/call_m_supervisor/description/bot/cameras_description.urdf.xacro (robot description, xacro)
@@ -2,36 +2,92 @@
 <robot name="bot" xmlns:xacro="http://ros.org/wiki/xacro">
 	<!-- THIS FILE NEED TO BE INCLUDED IN 'bot_description.urdf.xacro' -->
+	<!-- Copied from:  zed_wrapper/urdf/zed_macro.urdf.xacro-->
+	<xacro:include filename="$(find zed_wrapper)/urdf/include/materials.urdf.xacro" />
+	<xacro:property name="M_PI"     value="3.1415926535897931" />
 	<!--
-		////////////////////////
-		//////2 CAMERAS////////
-		///////////////////////
+		Parameters:
+		- name: the camera's name.  should match the parameter sent to the launch file for this camera
+		- model: the tye of camera, one of zed, zedm, zed2, zed2i
 	-->
-	<!--CAMERA 1 : FRONT-->
-	<link name="cam1_link">
+	<xacro:macro name="zed_camera" params="name=zed model=zed x=0.0 y=0.0 z=0.0 rot_z=0.0">
+		<xacro:property name="baseline" value="0.06" />
+		<xacro:property name="height" value="0.0265" />
+		<xacro:property name="bottom_slope" value="0.0" />
+		<xacro:property name="screw_offset_x" value="0.0" />
+		<xacro:property name="screw_offset_z" value="0.0" />
+		<xacro:property name="optical_offset_x" value="0.0" />
+		<!-- Camera mounting point (the threaded screw hole in the bottom) -->
+		<link name="${name}_link">
+			<visual>
+			<origin xyz="0 0 0" rpy="0 0 0"/>
+			<geometry>
+				<box size="0.0151 0.131 0.023"/>
+			</geometry>
+			</visual>
+			<inertial>
+			<origin xyz="0 0 0" rpy="0 0 0"/>
+			<mass value="0.035"/>
+			<inertia ixx="0.001"  ixy="0"  ixz="0" iyy="0.001" iyz="0" izz="0.001" />
+			</inertial>
+		</link>
+		<joint name="${name}_joint" type="continuous">
+			<parent link="base3_link"/>
+			<child link="${name}_link"/>
+			<origin xyz="${x} ${y} ${z}" rpy="0.0 0.0 ${rot_z}"/>
+			<axis xyz="0 1 0"/>
+		</joint>
+		<!-- Camera Center -->
+		<link name="${name}_camera_center">
 		<visual>
-		<origin xyz="0 0 0" rpy="0 0 0"/>
-		<geometry>
+			<origin xyz="${screw_offset_x} 0 ${screw_offset_z}" rpy="0 0 0"/>
+			<geometry>
+			<!--<mesh filename="package://zed_interfaces/meshes/${model}.stl" />-->
 			<box size="0.015 0.130 0.022"/>
-		</geometry>
+			</geometry>
+			<material name="${model}_mat" />
 		</visual>
 		<collision>
-		<origin xyz="0 0 0" rpy="0 0 0"/>
-		<geometry>
+			<geometry>
+			<!--<mesh filename="package://zed_interfaces/meshes/${model}.stl" />-->
 			<box size="0.015 0.130 0.022"/>
-		</geometry>
+			</geometry>
 		</collision>
-		<inertial>
-		<origin xyz="0 0 0" rpy="0 0 0"/>
-		<mass value="0.035"/>
-		<inertia ixx="0.001"  ixy="0"  ixz="0" iyy="0.001" iyz="0" izz="0.001" />
-		</inertial>
-	</link>
-	<joint name="cam1_joint" type="continuous">
-		<parent link="base3_link"/>
-		<child link="cam1_link"/>
-		<origin xyz="${(square1_length/2)+0.015/2} 0.0 ${(square3_height/2)-0.03-0.022/2}" rpy="0.0 0.0 0.0"/>
-		<axis xyz="0 1 0"/>
-	</joint>
-	<!--depth sensor-->
+		</link>
+		<joint name="${name}_camera_center_joint" type="fixed">
+		<parent link="${name}_link"/>
+		<child link="${name}_camera_center"/>
+		<origin xyz="0 0 0" rpy="0 ${bottom_slope} 0" />
+		</joint>
+		<!-- Left Camera -->
+		<link name="${name}_left_camera_frame" />
+		<joint name="${name}_left_camera_joint" type="fixed">
+		<parent link="${name}_camera_center"/>
+		<child link="${name}_left_camera_frame"/>
+		<origin xyz="${optical_offset_x} ${baseline/2} 0" rpy="0 0 0" />
+		</joint>
+		<link name="${name}_left_camera_optical_frame"/>
+		<joint name="${name}_left_camera_optical_joint" type="fixed">
+		<origin xyz="0 0 0" rpy="-${M_PI/2} 0.0 -${M_PI/2}"/>
+		<parent link="${name}_left_camera_frame"/>
+		<child link="${name}_left_camera_optical_frame"/>
+		</joint>
+		<!-- Right Camera -->
+		<link name="${name}_right_camera_frame" />
+		<joint name="${name}_right_camera_joint" type="fixed">
+		<parent link="${name}_camera_center"/>
+		<child link="${name}_right_camera_frame"/>
+		<origin xyz="${optical_offset_x} -${baseline/2} 0" rpy="0 0 0" />
+		</joint>
+		<link name="${name}_right_camera_optical_frame"/>
+		<joint name="${name}_right_camera_optical_joint" type="fixed">
+		<origin xyz="0 0 0" rpy="-${M_PI/2} 0.0 -${M_PI/2}"/>
+		<parent link="${name}_right_camera_frame"/>
+		<child link="${name}_right_camera_optical_frame"/>
+		</joint>
+	</xacro:macro>
+	<xacro:zed_camera name="cam1" model="zedm" x="${(square1_length/2)+0.015/2}" y="0.0" z="${(square3_height/2)-0.03-0.022/2}" rot_z="0.0"/>
+	<xacro:zed_camera name="cam2" model="zedm" x="${-((square1_length/2)+0.015/2)}" y="0.0" z="${(square3_height/2)-0.03-0.022/2}" rot_z="${M_PI}"/>
+	<!-- DEPTH sensors, not working in xacro-->
+	<!--CAMERA1 FRONT-->
 	<link name="cam1_depth_frame"/>
 	<joint name="cam1_depth_joint" type="fixed">
@@ -92,31 +148,5 @@
 		</sensor>
 	</gazebo>
-	<!--CAMERA 2 : BACK-->
-	<link name="cam2_link">
-		<visual>
-		<origin xyz="0 0 0" rpy="0 0 0"/>
-		<geometry>
-			<box size="0.015 0.130 0.022"/>
-		</geometry>
-		</visual>
-		<collision>
-		<origin xyz="0 0 0" rpy="0 0 0"/>
-		<geometry>
-			<box size="0.015 0.130 0.022"/>
-		</geometry>
-		</collision>
-		<inertial>
-		<origin xyz="0 0 0" rpy="0 0 0"/>
-		<mass value="0.035"/>
-		<inertia ixx="0.001"  ixy="0"  ixz="0" iyy="0.001" iyz="0" izz="0.001" />
-		</inertial>
-	</link>
-	<joint name="cam2_joint" type="continuous">
-		<parent link="base3_link"/>
-		<child link="cam2_link"/>
-		<origin xyz="${-((square1_length/2)+0.015/2)} 0.0 ${(square3_height/2)-0.03-0.022/2}" rpy="0.0 0.0 ${pi}"/>
-		<axis xyz="0 1 0"/>
-	</joint>
-	<!--depth sensor-->
+	<!--CAMERA2 BACK-->
 	<link name="cam2_depth_frame"/>
 	<joint name="cam2_depth_joint" type="fixed">

Commit message: Update

File: robot_ws_ros2/src/call_m_supervisor/description/bot/bot_description.urdf.xacro (robot description, xacro)
@@ -2,14 +2,15 @@
 <robot name="bot" xmlns:xacro="http://ros.org/wiki/xacro">
 	<!-- Define robot constants -->
-	<!-- Id changed, check also 'simu_bot_driver.cpp' -->
+	<!-- If changed, check also 'simu_bot_driver.cpp' for publish_command() -->
+	<!-- If need to change orientation, just change wheels, see wheels positions below + check lidars posiions and orientation in 'lidars_description.urdf.xacro'-->
 	<xacro:property name="square1_length" value="0.48"/>
 	<xacro:property name="square1_height" value="0.03"/>
-	<xacro:property name="square2_length" value="0.27"/>
-	<xacro:property name="square2_height" value="0.12"/>
+	<xacro:property name="square2_length" value="0.277"/>
+	<xacro:property name="square2_height" value="0.072"/>
 	<xacro:property name="square3_height" value="0.36"/>
 	<xacro:property name="wheels_radius" value="0.05"/>
 	<xacro:property name="triangle_lenght" value="0.32"/> <!-- Side's Triangle length-->
 	<xacro:property name="wheels_distance" value="${sqrt(((3*(triangle_lenght**4))/16)+((triangle_lenght**2)/4))}"/> <!-- Radius between origin and wheels-->
-	<xacro:property name="wheels_zoffset" value="0.02"/>
+	<xacro:property name="wheels_zoffset" value="0.03"/>
 	<!-- Define some commonly used intertial properties  -->
 	<xacro:macro name="box_inertia" params="m w h d">
@@ -186,7 +187,7 @@
 		</joint>
 	</xacro:macro>
-	<xacro:wheel prefix="wheel_2" angle="${-pi/2}" type="sphere" />
-	<xacro:wheel prefix="wheel_3" angle="${(2*pi/3)-pi/2}" type="sphere" />
-	<xacro:wheel prefix="wheel_1" angle="${(-2*pi/3)-pi/2}" type="sphere" />
+	<xacro:wheel prefix="wheel_2" angle="${pi}" type="sphere" />
+	<xacro:wheel prefix="wheel_3" angle="${(2*pi/3)+pi}" type="sphere" />
+	<xacro:wheel prefix="wheel_1" angle="${(-2*pi/3)+pi}" type="sphere" />
 	<xacro:include filename="lidars_description.urdf.xacro"/>
 	<xacro:include filename="cameras_description.urdf.xacro"/>

File: robot_ws_ros2/src/call_m_supervisor/description/bot/lidars_description.urdf.xacro (robot description, xacro)
@@ -13,5 +13,5 @@
 			<origin xyz="0 0 0" rpy="0 0 0"/>
 			<geometry>
-				<cylinder radius="0.0508" length="${0.1}"/>
+				<cylinder radius="0.0508" length="${0.05}"/>
 			</geometry>
 			</collision>
@@ -67,5 +67,5 @@
 		</gazebo>
 	</xacro:macro>
-	<xacro:lidar prefix="lidar1" x="${(square1_length/2)-0.0508}" y="${-((square1_length/2)-0.0508)}" alpha="${3*pi/4}" />
-	<xacro:lidar prefix="lidar2" x="${-((square1_length/2)-0.0508)}" y="${(square1_length/2)-0.0508}" alpha="${-pi/4}" />
+	<xacro:lidar prefix="lidar1" x="${-((square1_length/2)-0.0508)}" y="${-((square1_length/2)-0.0508)}" alpha="${pi/4}" />
+	<xacro:lidar prefix="lidar2" x="${(square1_length/2)-0.0508}" y="${(square1_length/2)-0.0508}" alpha="${-3*pi/4}" />
 </robot>

File: robot_ws_ros2/src/call_m_supervisor/description/bot/ros2_control.xacro (robot description, xacro)
@@ -58,5 +58,5 @@
     <gazebo>
     <plugin filename="libgazebo_ros2_control.so" name="gazebo_ros2_control">
-        <parameters>$(find call_m_supervisor)/config/controllers.yaml</parameters>
+        <parameters>$(find call_m_simulation)/config/controllers.yaml</parameters>
     </plugin>
     </gazebo>

Commit message: Update

File: robot_ws_ros2/src/call_m_supervisor/description/bot/bot_description.urdf.xacro (robot description, xacro)
@@ -59,4 +59,27 @@
 		<xacro:box_inertia m="15" w="${square1_length}" d="${square1_length}" h="${square1_height}"/>
 	</link>
+	<!-- Robot Support, to be deleted want controlling TDM MDP -->
+	<link name="base_sup_link">
+		<visual>
+		<geometry>
+			<cylinder radius="${wheels_radius}" length="${wheels_radius+wheels_zoffset+0.1}"/>
+		</geometry>
+		<material name="Cyan">
+			<color rgba="0 1.0 1.0 1.0"/>
+		</material>
+		</visual>
+		<collision>
+		<origin xyz="0 0 0" rpy="0 0 0"/>
+		<geometry>
+			<cylinder radius="${wheels_radius}" length="${wheels_radius*2}"/>
+		</geometry>
+		</collision>
+		<xacro:cylinder_inertia m="20" r="${wheels_radius}" h="${wheels_radius+wheels_zoffset+0.1}"/>
+	</link>
+	<joint name="$base_sup_joint" type="fixed">
+		<parent link="base_link"/>
+		<child link="base_sup_link"/>
+		<origin xyz="0.0 0.0 ${-((wheels_radius+wheels_zoffset+0.1)/2+(square1_height/2))}" rpy="0 0 0"/>
+	</joint>
 	<!-- Others Robot structures -->
 	<link name="base2_link">

File: robot_ws_ros2/src/call_m_supervisor/description/bot/ros2_control.xacro (robot description, xacro)
@@ -56,4 +56,5 @@
     </ros2_control>
     <!--we set up gazebo tag to indicate that we use ros2 control, a controller manager is integrated in it, so we need to indicate wich controller to use in yaml file-->
+    <!-- MDP / TDM : waitin ffor problem to be solve: https://github.com/ros-controls/gazebo_ros2_control/issues/295
     <gazebo>
     <plugin filename="libgazebo_ros2_control.so" name="gazebo_ros2_control">
@@ -61,3 +62,4 @@
     </plugin>
     </gazebo>
+    -->
 </robot>

Commit message: Update

File: robot_ws_ros2/src/call_m_supervisor/description/bot/bot_description.urdf.xacro (robot description, xacro)
@@ -59,27 +59,4 @@
 		<xacro:box_inertia m="15" w="${square1_length}" d="${square1_length}" h="${square1_height}"/>
 	</link>
-	<!-- Robot Support, to be deleted want controlling TDM MDP -->
-	<link name="base_sup_link">
-		<visual>
-		<geometry>
-			<cylinder radius="${wheels_radius}" length="${wheels_radius+wheels_zoffset+0.1}"/>
-		</geometry>
-		<material name="Cyan">
-			<color rgba="0 1.0 1.0 1.0"/>
-		</material>
-		</visual>
-		<collision>
-		<origin xyz="0 0 0" rpy="0 0 0"/>
-		<geometry>
-			<cylinder radius="${wheels_radius}" length="${wheels_radius*2}"/>
-		</geometry>
-		</collision>
-		<xacro:cylinder_inertia m="20" r="${wheels_radius}" h="${wheels_radius+wheels_zoffset+0.1}"/>
-	</link>
-	<joint name="$base_sup_joint" type="fixed">
-		<parent link="base_link"/>
-		<child link="base_sup_link"/>
-		<origin xyz="0.0 0.0 ${-((wheels_radius+wheels_zoffset+0.1)/2+(square1_height/2))}" rpy="0 0 0"/>
-	</joint>
 	<!-- Others Robot structures -->
 	<link name="base2_link">

File: robot_ws_ros2/src/call_m_supervisor/description/bot/cameras_description.urdf.xacro (robot description, xacro)
@@ -112,8 +112,8 @@
 		<update_rate>30.0</update_rate>
 		<camera name="cam1_cam">
-			<horizontal_fov>1.6</horizontal_fov>
+			<horizontal_fov>1.57</horizontal_fov>
 			<image>
-			<width>800</width>
-			<height>800</height>
+			<width>400</width>
+			<height>400</height>
 			<format>R8G8B8</format>
 			</image>
@@ -171,8 +171,8 @@
 		<update_rate>30.0</update_rate>
 		<camera name="cam2_cam">
-			<horizontal_fov>1.6</horizontal_fov>
+			<horizontal_fov>1.57</horizontal_fov>
 			<image>
-			<width>800</width>
-			<height>800</height>
+			<width>400</width>
+			<height>400</height>
 			<format>R8G8B8</format>
 			</image>

File: robot_ws_ros2/src/call_m_supervisor/description/bot/ros2_control.xacro (robot description, xacro)
@@ -56,5 +56,5 @@
     </ros2_control>
     <!--we set up gazebo tag to indicate that we use ros2 control, a controller manager is integrated in it, so we need to indicate wich controller to use in yaml file-->
-    <!-- MDP / TDM : waitin ffor problem to be solve: https://github.com/ros-controls/gazebo_ros2_control/issues/295
+    <!-- MDP / TDM : waitin ffor problem to be solve: https://github.com/ros-controls/gazebo_ros2_control/issues/295 -->
     <gazebo>
     <plugin filename="libgazebo_ros2_control.so" name="gazebo_ros2_control">
@@ -62,4 +62,3 @@
     </plugin>
     </gazebo>
-    -->
 </robot>

Commit message: Update

File: robot_ws_ros2/src/call_m_supervisor/description/bot/bot_description.urdf.xacro (robot description, xacro)
@@ -9,4 +9,6 @@
 	<xacro:property name="square2_height" value="0.072"/>
 	<xacro:property name="square3_height" value="0.36"/>
+	<xacro:property name="support1_width" value="0.26"/>
+	<xacro:property name="support2_height" value="0.33"/>
 	<xacro:property name="wheels_radius" value="0.05"/>
 	<xacro:property name="triangle_lenght" value="0.32"/> <!-- Side's Triangle length-->
@@ -80,4 +82,46 @@
 		<child link="base2_link"/>
 		<origin xyz="0.0 0.0 ${(square1_height/2)+(square2_height/2)}" rpy="0 0 0"/>
+	</joint>
+	<link name="support1_link">
+		<visual>
+		<geometry>
+			<box size="${square1_length} ${support1_width} ${square1_height}"/>
+		</geometry>
+		<material name="Cyan">
+			<color rgba="0 1.0 1.0 1.0"/>
+		</material>
+		</visual>
+		<collision>
+		<geometry>
+			<box size="${square1_length} ${support1_width} ${square1_height}"/>
+		</geometry>
+		</collision>
+		<xacro:box_inertia m="0.5" w="${square1_length}" d="${support1_width}" h="${square1_height}"/>
+	</link>
+	<joint name="support1_joint" type="fixed">
+		<parent link="base3_link"/>
+		<child link="support1_link"/>
+		<origin xyz="0.0 ${square1_length/2 + support1_width/2} ${square1_height/2 - square3_height/2}" rpy="0 0 0"/>
+	</joint>
+	<link name="support2_link">
+		<visual>
+		<geometry>
+			<box size="${square1_length} ${square1_height} ${support2_height}"/>
+		</geometry>
+		<material name="Cyan">
+			<color rgba="0 1.0 1.0 1.0"/>
+		</material>
+		</visual>
+		<collision>
+		<geometry>
+			<box size="${square1_length} ${square1_height} ${support2_height}"/>
+		</geometry>
+		</collision>
+		<xacro:box_inertia m="0.5" w="${square1_length}" d="${square1_height}" h="${support2_height}"/>
+	</link>
+	<joint name="support2_joint" type="fixed">
+		<parent link="support1_link"/>
+		<child link="support2_link"/>
+		<origin xyz="0.0 ${support1_width/2 - square1_height/2} ${support2_height/2 + square1_height/2}" rpy="0 0 0"/>
 	</joint>
 	<link name="base3_link">
