Commit message: Merged arm and call-m URDFs with their respective controllers working, and deleted the comments on the .xacro files

File: robot_ws_ros2/src/call_m_supervisor/urdf/cameras_description.urdf.xacro (robot description, xacro)
@@ -1,13 +1,6 @@
 <?xml version="1.0"?>
 <robot name="bot" xmlns:xacro="http://ros.org/wiki/xacro">
-	<!-- THIS FILE NEED TO BE INCLUDED IN 'bot_description.urdf.xacro' -->
-	<!-- Copied from:  zed_wrapper/urdf/zed_macro.urdf.xacro-->
 	<xacro:include filename="$(find zed_wrapper)/urdf/include/materials.urdf.xacro" />
 	<xacro:property name="M_PI"     value="3.1415926535897931" />
-	<!--
-		Parameters:
-		- name: the camera's name.  should match the parameter sent to the launch file for this camera
-		- model: the tye of camera, one of zed, zedm, zed2, zed2i
-	-->
 	<xacro:macro name="zed_camera" params="name=zed model=zed x=0.0 y=0.0 z=0.0 rot_z=0.0">
 		<xacro:property name="baseline" value="0.06" />
@@ -17,5 +10,4 @@
 		<xacro:property name="screw_offset_z" value="0.0" />
 		<xacro:property name="optical_offset_x" value="0.0" />
-		<!-- Camera mounting point (the threaded screw hole in the bottom) -->
 		<link name="${name}_camera_link">
 			<visual>
@@ -37,10 +29,8 @@
 			<axis xyz="0 1 0"/>
 		</joint>
-		<!-- Camera Center -->
 		<link name="${name}_camera_center">
 		<visual>
 			<origin xyz="${screw_offset_x} 0 ${screw_offset_z}" rpy="0 0 0"/>
 			<geometry>
-			<!--<mesh filename="package://zed_interfaces/meshes/${model}.stl" />-->
 			<box size="0.015 0.130 0.022"/>
 			</geometry>
@@ -49,5 +39,4 @@
 		<collision>
 			<geometry>
-			<!--<mesh filename="package://zed_interfaces/meshes/${model}.stl" />-->
 			<box size="0.015 0.130 0.022"/>
 			</geometry>
@@ -59,5 +48,4 @@
 		<origin xyz="0 0 0" rpy="0 ${bottom_slope} 0" />
 		</joint>
-		<!-- Left Camera -->
 		<link name="${name}_left_camera_frame" />
 		<joint name="${name}_left_camera_joint" type="fixed">
@@ -72,5 +60,4 @@
 		<child link="${name}_left_camera_optical_frame"/>
 		</joint>
-		<!-- Right Camera -->
 		<link name="${name}_right_camera_frame" />
 		<joint name="${name}_right_camera_joint" type="fixed">
@@ -85,18 +72,7 @@
 		<child link="${name}_right_camera_optical_frame"/>
 		</joint>
-		<!-- IMU -->
-		<!--
-		<link name="${name}_imu_link"/>
-		<joint name="${name}_imu_link_joint" type="fixed">
-		<origin xyz="0 0 0" rpy="0.0 0.0 0.0"/>
-		<parent link="${name}_camera_center"/>
-		<child link="${name}_imu_link"/>
-		</joint>
-		-->
 	</xacro:macro>
 	<xacro:zed_camera name="cam1" model="zedm" x="${(square1_length/2)+0.015/2}" y="0.0" z="${(square3_height/2)-0.03-0.022/2}" rot_z="0.0"/>
 	<xacro:zed_camera name="cam2" model="zedm" x="${-((square1_length/2)+0.015/2)}" y="0.0" z="${(square3_height/2)-0.03-0.022/2}" rot_z="${M_PI}"/>
-	<!-- DEPTH sensors, not working in xacro-->
-	<!--CAMERA1 FRONT-->
 	<link name="cam1_depth_frame"/>
 	<joint name="cam1_depth_joint" type="fixed">
@@ -106,6 +82,4 @@
 	</joint>
 	<gazebo reference="cam1_camera_link">
-		<!-- Gazebo is unable to use the same <material> tags that are already in the URDF (that RViz uses). -->
-    	<!-- Instead, we need to add gazebo tags for our links that refer to Gazebo materials -->
         <material>Gazebo/Orange</material>
 		<sensor type="depth" name="cam1">
@@ -129,5 +103,4 @@
 		</camera>
 		<plugin name="depth_camera_controller" filename="libgazebo_ros_camera.so">
-			<!--/cam1/zed_node/rgb/image_rect_color-->
 		    <ros>
                 <namespace>cam1</namespace>
@@ -157,5 +130,4 @@
 		</sensor>
 	</gazebo>
-	<!--CAMERA2 BACK-->
 	<link name="cam2_depth_frame"/>
 	<joint name="cam2_depth_joint" type="fixed">
@@ -165,6 +137,4 @@
 	</joint>
 	<gazebo reference="cam2_camera_link">
-		<!-- Gazebo is unable to use the same <material> tags that are already in the URDF (that RViz uses). -->
-    	<!-- Instead, we need to add gazebo tags for our links that refer to Gazebo materials -->
         <material>Gazebo/Orange</material>
 		<sensor type="depth" name="cam2">

File: robot_ws_ros2/src/call_m_supervisor/urdf/imu_description.urdf.xacro (robot description, xacro)
@@ -1,5 +1,4 @@
 <?xml version="1.0"?>
 <robot name="bot" xmlns:xacro="http://ros.org/wiki/xacro">
-	<!-- THIS FILE NEED TO BE INCLUDED IN 'bot_description.urdf.xacro' -->
     <link name="imu_link">
     <visual>
@@ -60,5 +59,4 @@
         </angular_velocity>
         <linear_acceleration>
-        <!--If values are noisy: https://answers.gazebosim.org//question/810/is-it-possible-to-reduce-inertial-sensor-noise-by-adjusting-gazebo-parameters/-->
             <x>
             <noise type="gaussian">

File: robot_ws_ros2/src/call_m_supervisor/urdf/ros2_control.xacro (robot description, xacro)
@@ -1,5 +1,4 @@
 <?xml version="1.0"?>
 <robot name="bot" xmlns:xacro="http://ros.org/wiki/xacro">
-    <!--we specify joints that will be controlled-->
     <ros2_control name="GazeboSystem" type="system">
         <hardware>
@@ -55,6 +54,4 @@
         </joint>
     </ros2_control>
-    <!--we set up gazebo tag to indicate that we use ros2 control, a controller manager is integrated in it, so we need to indicate wich controller to use in yaml file-->
-    <!--Update problem (solved): https://github.com/ros-controls/gazebo_ros2_control/issues/295 -->
     <gazebo>
     <plugin filename="libgazebo_ros2_control.so" name="gazebo_ros2_control">

File: robot_ws_ros2/src/call_m_supervisor/urdf/sim.urdf.xacro (robot description, xacro)
@@ -1,4 +1,242 @@
 <?xml version="1.0"?>
 <robot xmlns:xacro="http://wiki.ros.org/xacro" name="call_m_arm">
+  	<!-- Define robot constants -->
+	<!-- If changed, check also 'simu_bot_driver.cpp' for publish_command() -->
+	<!-- If need to change orientation, just change wheels, see wheels positions below + check lidars posiions and orientation in 'lidars_description.urdf.xacro'-->
+	<xacro:property name="square1_length" value="0.48"/>
+	<xacro:property name="square1_height" value="0.03"/>
+	<xacro:property name="square2_length" value="0.277"/>
+	<xacro:property name="square2_height" value="0.072"/>
+	<xacro:property name="square3_height" value="0.36"/>
+	<xacro:property name="support1_width" value="0.26"/>
+	<xacro:property name="support2_height" value="0.33"/>
+	<xacro:property name="wheels_radius" value="0.05"/>
+	<xacro:property name="triangle_lenght" value="0.32"/> <!-- Side's Triangle length-->
+	<xacro:property name="wheels_distance" value="${sqrt(((3*(triangle_lenght**4))/16)+((triangle_lenght**2)/4))}"/> <!-- Radius between origin and wheels-->
+	<xacro:property name="wheels_zoffset" value="0.03"/>
+	<!-- Define some commonly used intertial properties  -->
+	<xacro:macro name="box_inertia" params="m w h d">
+		<inertial>
+		<origin xyz="0 0 0" rpy="${pi/2} 0 ${pi/2}"/>
+		<mass value="${m}"/>
+		<inertia ixx="${(m/12) * (h*h + d*d)}" ixy="0.0" ixz="0.0" iyy="${(m/12) * (w*w + d*d)}" iyz="0.0" izz="${(m/12) * (w*w + h*h)}"/>
+		</inertial>
+	</xacro:macro>
+	<xacro:macro name="cylinder_inertia" params="m r h">
+		<inertial>
+		<origin xyz="0 0 0" rpy="${pi/2} 0 0" />
+		<mass value="${m}"/>
+		<inertia ixx="${(m/12) * (3*r*r + h*h)}" ixy = "0" ixz = "0" iyy="${(m/12) * (3*r*r + h*h)}" iyz = "0" izz="${(m/2) * (r*r)}"/>
+		</inertial>
+	</xacro:macro>
+	<xacro:macro name="sphere_inertia" params="m r">
+		<inertial>
+		<mass value="${m}"/>
+		<inertia ixx="${(2/5) * m * (r*r)}" ixy="0.0" ixz="0.0" iyy="${(2/5) * m * (r*r)}" iyz="0.0" izz="${(2/5) * m * (r*r)}"/>
+		</inertial>
+	</xacro:macro>
+	<!-- Robot Base -->
+	<!-- Dummy link may need to be added because KDL does not support root link with inertia. But simulation not working with it-->
+	<!--<link name="dummy"></link>
+	<joint name="init_joint" type="fixed">
+		<parent link="dummy"/>
+		<child link="base_link"/>
+		<origin xyz="0.0 0.0 ).0}" rpy="0 0 0"/>
+	</joint>
+	-->
+	<link name="base_link">
+		<visual>
+		<geometry>
+			<box size="${square1_length} ${square1_length} ${square1_height}"/>
+		</geometry>
+		<material name="Cyan">
+			<color rgba="0 1.0 1.0 1.0"/>
+		</material>
+		</visual>
+		<collision>
+		<geometry>
+			<box size="${square1_length} ${square1_length} ${square1_height}"/>
+		</geometry>
+		</collision>
+		<xacro:box_inertia m="15" w="${square1_length}" d="${square1_length}" h="${square1_height}"/>
+	</link>
+	<!-- Others Robot structures -->
+	<link name="base2_link">
+		<visual>
+		<geometry>
+			<box size="${square2_length} ${square2_length} ${square2_height}"/>
+		</geometry>
+		<material name="Cyan">
+			<color rgba="0 1.0 1.0 1.0"/>
+		</material>
+		</visual>
+		<collision>
+		<geometry>
+			<box size="${square2_length} ${square2_length} ${square2_height*0.8}"/>
+		</geometry>
+		</collision>
+		<xacro:box_inertia m="0.5" w="${square2_length}" d="${square2_length}" h="${square2_height}"/>
+	</link>
+	<joint name="base2_joint" type="fixed">
+		<parent link="base_link"/>
+		<child link="base2_link"/>
+		<origin xyz="0.0 0.0 ${(square1_height/2)+(square2_height/2)}" rpy="0 0 0"/>
+	</joint>
+	<link name="support1_link">
+		<visual>
+		<geometry>
+			<box size="${square1_length} ${support1_width} ${square1_height}"/>
+		</geometry>
+		<material name="Cyan">
+			<color rgba="0 1.0 1.0 1.0"/>
+		</material>
+		</visual>
+		<collision>
+		<geometry>
+			<box size="${square1_length} ${support1_width} ${square1_height}"/>
+		</geometry>
+		</collision>
+		<xacro:box_inertia m="0.5" w="${square1_length}" d="${support1_width}" h="${square1_height}"/>
+	</link>
+	<joint name="support1_joint" type="fixed">
+		<parent link="base3_link"/>
+		<child link="support1_link"/>
+		<origin xyz="0.0 ${square1_length/2 + support1_width/2} ${square1_height/2 - square3_height/2}" rpy="0 0 0"/>
+	</joint>
+	<link name="support2_link">
+		<visual>
+		<geometry>
+			<box size="${square1_length} ${square1_height} ${support2_height}"/>
+		</geometry>
+		<material name="Cyan">
+			<color rgba="0 1.0 1.0 1.0"/>
+		</material>
+		</visual>
+		<collision>
+		<geometry>
+			<box size="${square1_length} ${square1_height} ${support2_height}"/>
+		</geometry>
+		</collision>
+		<xacro:box_inertia m="0.5" w="${square1_length}" d="${square1_height}" h="${support2_height}"/>
+	</link>
+	<joint name="support2_joint" type="fixed">
+		<parent link="support1_link"/>
+		<child link="support2_link"/>
+		<origin xyz="0.0 ${support1_width/2 - square1_height/2} ${support2_height/2 + square1_height/2}" rpy="0 0 0"/>
+	</joint>
+	<link name="base3_link">
+		<visual>
+		<geometry>
+			<box size="${square1_length} ${square1_length} ${square3_height}"/>
+		</geometry>
+		<material name="Cyan">
+			<color rgba="0 1.0 1.0 1.0"/>
+		</material>
+		</visual>
+		<collision>
+		<geometry>
+			<box size="${square1_length} ${square1_length} ${square3_height}"/>
+		</geometry>
+		</collision>
+		<xacro:box_inertia m="0.5" w="${square1_length}" d="${square1_length}" h="${square3_height}"/>
+	</link>
+	<joint name="base3_joint" type="fixed">
+		<parent link="base_link"/>
+		<child link="base3_link"/>
+		<origin xyz="0.0 0.0 ${(square1_height/2)+square2_height+(square3_height/2)}" rpy="0 0 0"/>
+	</joint>
+	<link name="base4_link">
+		<visual>
+		<geometry>
+			<box size="${square1_length/4} ${square1_length/30} ${0.04}"/>
+		</geometry>
+		<material name="Green">
+			<color rgba="1.0 0.0 1.0 1.0"/>
+		</material>
+		</visual>
+	</link>
+	<joint name="base4_joint" type="fixed">
+		<parent link="base3_link"/>
+		<child link="base4_link"/>
+		<origin xyz="${square1_length/2-square1_length/4} 0.0 ${(square3_height/2)+0.02}" rpy="0 0 0"/>
+	</joint>
+	<!-- Robot Footprint-->
+	<link name="base_footprint">
+		<xacro:box_inertia m="0" w="0" d="0" h="0"/>
+	</link>
+	<joint name="base_joint" type="fixed">
+		<parent link="base_link"/>
+		<child link="base_footprint"/>
+		<origin xyz="0.0 0.0 ${-(wheels_radius*2+wheels_zoffset+square1_height/2)}" rpy="0 0 0"/>
+	</joint>
+	  <!-- 3 Wheels and there support to simulate sphere joint -->
+	<xacro:macro name="wheel" params="prefix angle type">
+		<!--wheel support-->
+		<link name="${prefix}_sup_link">
+		<visual>
+			<geometry>
+				<cylinder radius="${wheels_radius}" length="${wheels_zoffset}"/>
+			</geometry>
+			<material name="Gray">
+			<color rgba="0.5 0.5 0.5 1.0"/>
+			</material>
+		</visual>
+		<collision>
+			<geometry>
+			<cylinder radius="${wheels_radius}" length="${wheels_zoffset/2}"/>
+			</geometry>
+		</collision>
+		<xacro:cylinder_inertia m="2" r="${wheels_radius}" h="${wheels_zoffset}"/>
+		</link>
+		<joint name="${prefix}_sup_joint" type="continuous">
+			<parent link="base_link"/>
+			<child link="${prefix}_sup_link"/>
+			<origin xyz="${wheels_distance*cos(angle)} ${wheels_distance*sin(angle)} ${-((wheels_zoffset/2)+(square1_height/2))}" rpy="0 0 0"/>
+			<axis xyz="0 0 1"/>
+		</joint>
+		<!--wheel-->
+		<link name="${prefix}_link">
+		<visual>
+			<geometry>
+				<sphere radius="${wheels_radius}"/>
+			</geometry>
+			<material name="Gray">
+			<color rgba="0.5 0.5 0.5 1.0"/>
+			</material>
+		</visual>
+		<xacro:if value="${type == 'sphere'}">
+			<collision>
+			<origin xyz="0 0 0" rpy="0 0 0"/>
+			<geometry>
+				<sphere radius="${wheels_radius}"/>
+			</geometry>
+			</collision>
+			<xacro:sphere_inertia m="0.5" r="${wheels_radius}"/>
+		</xacro:if>
+		<xacro:if value="${type == 'cylinder'}">
+			<collision>
+			<origin xyz="0 0 0" rpy="${pi/2} 0 0"/>
+			<geometry>
+				<cylinder radius="${wheels_radius}" length="${wheels_radius*2}"/>
+			</geometry>
+			</collision>
+			<xacro:cylinder_inertia m="0.5" r="${wheels_radius}" h="${wheels_radius*2}"/>
+		</xacro:if>
+		</link>
+		<joint name="${prefix}_joint" type="continuous">
+			<parent link="${prefix}_sup_link"/>
+			<child link="${prefix}_link"/>
+			<origin xyz="0.0 0.0 ${-wheels_radius-wheels_zoffset/2}" rpy="0 0 0"/>
+			<axis xyz="0 1 0"/>
+		</joint>
+	</xacro:macro>
+	<xacro:wheel prefix="wheel_2" angle="${pi}" type="sphere" />
+	<xacro:wheel prefix="wheel_3" angle="${(2*pi/3)+pi}" type="sphere" />
+	<xacro:wheel prefix="wheel_1" angle="${(-2*pi/3)+pi}" type="sphere" />
+	<xacro:include filename="lidars_description.urdf.xacro"/>
+	<xacro:include filename="cameras_description.urdf.xacro"/>
+	<!--The simulated IMU seems to be noisy too much even with no noise set, so we don't use it for linear movement-->
+	<xacro:include filename="imu_description.urdf.xacro"/>
+	<xacro:include filename="gazebo_template.urdf.xacro"/>
    <!-- robot name parameter -->
    <xacro:arg name="name" default="ur"/>
@@ -49,40 +287,9 @@
    <!-- convert to property to use substitution in function -->
    <xacro:property name="initial_positions_file" default="$(arg initial_positions_file)"/>
-  <!-- world link-->
-    <link name="world" />
-   <!-- create link fixed to the "box-link" -->
-   <link name="box-link">
-    <visual>
-        <origin xyz="0 0 0" rpy="0 0 0"/>
-        <geometry>
-            <box size="0.8 0.6 0.64"/> <!-- 80x60x64 cm in meters -->
-        </geometry>
-        <material name="Grey">
-            <color rgba="0.5 0.5 0.5 1.0"/>
-        </material>
-    </visual>
-    <collision>
-        <origin xyz="0 0 0" rpy="0 0 0"/>
-        <geometry>
-            <box size="0.8 0.6 0.64"/>
-        </geometry>
-    </collision>
-    <inertial>
-        <mass value="5.0"/> <!-- Adjust mass as needed -->
-        <origin xyz="0 0 0" rpy="0 0 0"/>
-        <inertia ixx="0.1" ixy="0.0" ixz="0.0" iyy="0.1" iyz="0.0" izz="0.1"/> <!-- Adjust inertia as needed -->
-    </inertial>
-  </link>
-  <!-- World link and box joint-->
-  <joint name="world_to_box_base" type="fixed">
-    <origin xyz="0 0 0.32" rpy="0 0 0" />
-    <parent link="world" />
-    <child link="box-link" />
-  </joint>
    <!-- arm -->
    <xacro:ur_robot
      name="$(arg name)"
      tf_prefix="$(arg tf_prefix)"
-     parent="box-link"
+     parent="base_link"
      joint_limits_parameters_file="$(arg joint_limit_params)"
      kinematics_parameters_file="$(arg kinematics_params)"
@@ -120,23 +327,5 @@
      <origin xyz="0.14 0 0.32" rpy="0 0 1.57" />          <!-- position robot in the world -->
    </xacro:ur_robot>
-   <xacro:if value="$(arg sim_gazebo)">
-    <!-- Gazebo plugins -->
-    <gazebo>
-      <plugin filename="libgazebo_ros2_control.so" name="gazebo_ros2_control">
-        <parameters>$(arg simulation_controllers)</parameters>
-      </plugin>
-    </gazebo>
-  </xacro:if>
-  <xacro:if value="$(arg sim_ignition)">
-    <!-- Gazebo plugins -->
-    <gazebo reference="box-link">
-    </gazebo>
-    <gazebo>
-      <plugin filename="libign_ros2_control-system.so" name="ign_ros2_control::IgnitionROS2ControlPlugin">
-        <parameters>$(arg simulation_controllers)</parameters>
-        <controller_manager_node_name>$(arg tf_prefix)controller_manager</controller_manager_node_name>
-      </plugin>
-    </gazebo>
-  </xacro:if>
+	<xacro:include filename="ros2_control.xacro"/>
 <xacro:include filename="$(find call_m_arm_pkg)/urdf/fake_gripper.xacro"/>
 <xacro:fake_gripper parent_link="$(arg tf_prefix)tool0" gripper_x="0" gripper_y="0" gripper_z="0.0" gripper_roll="0" gripper_pitch="0" gripper_yaw="1.57"/>
