Commit message: Modified controller yaml files to support the arm and the robot, and changed the folder under which the urdf resources are

File: robot_ws_ros2/src/call_m_supervisor/urdf/sim.urdf.xacro (robot description, xacro)
@@ -9,5 +9,5 @@
    <xacro:arg name="ur_type" default="ur5e"/>
    <!-- parameters -->
-   <xacro:arg name="tf_prefix" default="" />
+   <xacro:arg name="tf_prefix" default="/ur5e/" />
    <xacro:arg name="joint_limit_params" default="$(find ur_description)/config/$(arg ur_type)/joint_limits.yaml"/>
    <xacro:arg name="kinematics_params" default="$(find ur_description)/config/$(arg ur_type)/default_kinematics.yaml"/>
@@ -122,6 +122,4 @@
    <xacro:if value="$(arg sim_gazebo)">
     <!-- Gazebo plugins -->
-    <gazebo reference="box-link">
-    </gazebo>
     <gazebo>
       <plugin filename="libgazebo_ros2_control.so" name="gazebo_ros2_control">
@@ -142,5 +140,5 @@
   </xacro:if>
 <xacro:include filename="$(find call_m_arm_pkg)/urdf/fake_gripper.xacro"/>
-<xacro:fake_gripper parent_link="tool0" gripper_x="0" gripper_y="0" gripper_z="0.0" gripper_roll="0" gripper_pitch="0" gripper_yaw="1.57"/>
+<xacro:fake_gripper parent_link="$(arg tf_prefix)tool0" gripper_x="0" gripper_y="0" gripper_z="0.0" gripper_roll="0" gripper_pitch="0" gripper_yaw="1.57"/>
   <link name="zed_eef_link">
     <visual>
@@ -164,5 +162,5 @@
   <!-- Joint connecting the bracket to the specified parent link -->
   <joint name="zed_eef_joint" type="fixed">
-    <parent link="tool0"/>
+    <parent link="$(arg tf_prefix)tool0"/>
     <child link="zed_eef_link"/>
     <origin rpy="0.785 0 1.57" xyz="-0.08 0 0"/>

Commit message: Fixed a bug where the eef couldnt be manually moved due to the namespace not being declared next to the joints

File: robot_ws_ros2/src/call_m_supervisor/urdf/sim.urdf.xacro (robot description, xacro)
@@ -3,10 +3,6 @@
 	<link name="world">
 	</link>
-	<joint name="world-base_link" type="fixed">
-		<parent link="world"/>
-		<child link="base_link"/>
-		<origin xyz="0.0 -1.0 0.2" rpy="0.0 0.0 0.0"/>
-	</joint>
-  	<!-- Define robot constants -->
+  	<!-- De
+	fine robot constants -->
 	<!-- If changed, check also 'simu_bot_driver.cpp' for publish_command() -->
 	<!-- If need to change orientation, just change wheels, see wheels positions below + check lidars posiions and orientation in 'lidars_description.urdf.xacro'-->
@@ -68,4 +64,9 @@
 		<xacro:box_inertia m="15" w="${square1_length}" d="${square1_length}" h="${square1_height}"/>
 	</link>
+		<joint name="world-base_link" type="fixed">
+		<parent link="world"/>
+		<child link="base_link"/>
+		<origin xyz="0.0 -1.0 0.2" rpy="0.0 0.0 0.0"/>
+	</joint>
 	<!-- Others Robot structures -->
 	<link name="base2_link">

Commit message: The simulated grasps now work with call-m original URDF

File: robot_ws_ros2/src/call_m_supervisor/urdf/sim.urdf.xacro (robot description, xacro)
@@ -64,5 +64,5 @@
 		<xacro:box_inertia m="15" w="${square1_length}" d="${square1_length}" h="${square1_height}"/>
 	</link>
-		<joint name="world-base_link" type="fixed">
+	<joint name="world-base_link" type="fixed">
 		<parent link="world"/>
 		<child link="base_link"/>
@@ -333,5 +333,5 @@
      trajectory_port="$(arg trajectory_port)"
      >
-     <origin xyz="0.14 0 0.32" rpy="0 0 1.57" />          <!-- position robot in the world -->
+     <origin xyz="0.0 0 0.44" rpy="0 0 1.57" />          <!-- position robot in the world -->
    </xacro:ur_robot>
 	<xacro:include filename="ros2_control.xacro"/>
