Commit message: Changed the controllers.yaml and other dependencies to adapt the new arm namespace

File: robot_ws_ros2/src/call_m_arm/call_m_moveit_config/srdf/ur.srdf.xacro (robot description, xacro)
@@ -4,5 +4,5 @@
   <xacro:arg name="name" default="ur"/>
   <!-- parameters -->
-  <xacro:arg name="prefix" default="" />
+  <xacro:arg name="prefix" default="ur5e/" />
   <xacro:include filename="$(find call_m_moveit_config)/srdf/ur_macro.srdf.xacro"/>
   <xacro:ur_srdf name="$(arg name)" prefix="$(arg prefix)"/>

File: robot_ws_ros2/src/call_m_arm/call_m_moveit_config/srdf/ur_macro.srdf.xacro (robot description, xacro)
@@ -74,36 +74,199 @@
     <!--VIRTUAL JOINT - Purpose - this element defines a virtual joint between a robot link and an external frame of reference (considered fixed with respect to the robot)-->
     <!--DISABLE COLLISIONS - By default it is assumed that any link of the robot could potentially come into collision with any other link in the robot. This tag disables collision checking between a specified pair of links. -->
-    <disable_collisions link1="base_link_inertia" link2="box-link" reason="Adjacent"/>
-    <disable_collisions link1="base_link_inertia" link2="shoulder_link" reason="Adjacent"/>
-    <disable_collisions link1="base_link_inertia" link2="zed_eef_link" reason="Never"/>
-    <disable_collisions link1="box-link" link2="shoulder_link" reason="Never"/>
+    <!--DISABLE COLLISIONS: By default it is assumed that any link of the robot could potentially come into collision with any other link in the robot. This tag disables collision checking between a specified pair of links. -->
+    <disable_collisions link1="base2_link" link2="base3_link" reason="Never"/>
+    <disable_collisions link1="base2_link" link2="base_link" reason="Adjacent"/>
+    <disable_collisions link1="base2_link" link2="cam1_camera_center" reason="Never"/>
+    <disable_collisions link1="base2_link" link2="cam2_camera_center" reason="Never"/>
+    <disable_collisions link1="base2_link" link2="imu_link" reason="Default"/>
+    <disable_collisions link1="base2_link" link2="lidar1_link" reason="Never"/>
+    <disable_collisions link1="base2_link" link2="lidar2_link" reason="Never"/>
+    <disable_collisions link1="base2_link" link2="support1_link" reason="Never"/>
+    <disable_collisions link1="base2_link" link2="support2_link" reason="Never"/>
+    <disable_collisions link1="base2_link" link2="ur5e/base_link_inertia" reason="Never"/>
+    <disable_collisions link1="base2_link" link2="ur5e/shoulder_link" reason="Never"/>
+    <disable_collisions link1="base2_link" link2="wheel_1_link" reason="Never"/>
+    <disable_collisions link1="base2_link" link2="wheel_1_sup_link" reason="Never"/>
+    <disable_collisions link1="base2_link" link2="wheel_2_link" reason="Never"/>
+    <disable_collisions link1="base2_link" link2="wheel_2_sup_link" reason="Never"/>
+    <disable_collisions link1="base2_link" link2="wheel_3_link" reason="Never"/>
+    <disable_collisions link1="base2_link" link2="wheel_3_sup_link" reason="Never"/>
+    <disable_collisions link1="base3_link" link2="base_link" reason="Adjacent"/>
+    <disable_collisions link1="base3_link" link2="cam1_camera_center" reason="Adjacent"/>
+    <disable_collisions link1="base3_link" link2="cam2_camera_center" reason="Adjacent"/>
+    <disable_collisions link1="base3_link" link2="imu_link" reason="Never"/>
+    <disable_collisions link1="base3_link" link2="lidar1_link" reason="Default"/>
+    <disable_collisions link1="base3_link" link2="lidar2_link" reason="Default"/>
+    <disable_collisions link1="base3_link" link2="support1_link" reason="Adjacent"/>
+    <disable_collisions link1="base3_link" link2="support2_link" reason="Never"/>
+    <disable_collisions link1="base3_link" link2="ur5e/base_link_inertia" reason="Default"/>
+    <disable_collisions link1="base3_link" link2="ur5e/shoulder_link" reason="Default"/>
+    <disable_collisions link1="base3_link" link2="ur5e/upper_arm_link" reason="Default"/>
+    <disable_collisions link1="base3_link" link2="wheel_1_link" reason="Never"/>
+    <disable_collisions link1="base3_link" link2="wheel_1_sup_link" reason="Never"/>
+    <disable_collisions link1="base3_link" link2="wheel_2_link" reason="Never"/>
+    <disable_collisions link1="base3_link" link2="wheel_2_sup_link" reason="Never"/>
+    <disable_collisions link1="base3_link" link2="wheel_3_link" reason="Never"/>
+    <disable_collisions link1="base3_link" link2="wheel_3_sup_link" reason="Never"/>
+    <disable_collisions link1="base_link" link2="cam1_camera_center" reason="Never"/>
+    <disable_collisions link1="base_link" link2="cam2_camera_center" reason="Never"/>
+    <disable_collisions link1="base_link" link2="imu_link" reason="Adjacent"/>
+    <disable_collisions link1="base_link" link2="lidar1_link" reason="Adjacent"/>
+    <disable_collisions link1="base_link" link2="lidar2_link" reason="Adjacent"/>
+    <disable_collisions link1="base_link" link2="support1_link" reason="Never"/>
+    <disable_collisions link1="base_link" link2="support2_link" reason="Never"/>
+    <disable_collisions link1="base_link" link2="ur5e/base_link_inertia" reason="Adjacent"/>
+    <disable_collisions link1="base_link" link2="ur5e/shoulder_link" reason="Never"/>
+    <disable_collisions link1="base_link" link2="wheel_1_link" reason="Never"/>
+    <disable_collisions link1="base_link" link2="wheel_1_sup_link" reason="Adjacent"/>
+    <disable_collisions link1="base_link" link2="wheel_2_link" reason="Never"/>
+    <disable_collisions link1="base_link" link2="wheel_2_sup_link" reason="Adjacent"/>
+    <disable_collisions link1="base_link" link2="wheel_3_link" reason="Never"/>
+    <disable_collisions link1="base_link" link2="wheel_3_sup_link" reason="Adjacent"/>
+    <disable_collisions link1="cam1_camera_center" link2="cam2_camera_center" reason="Never"/>
+    <disable_collisions link1="cam1_camera_center" link2="imu_link" reason="Never"/>
+    <disable_collisions link1="cam1_camera_center" link2="lidar1_link" reason="Never"/>
+    <disable_collisions link1="cam1_camera_center" link2="lidar2_link" reason="Never"/>
+    <disable_collisions link1="cam1_camera_center" link2="support1_link" reason="Never"/>
+    <disable_collisions link1="cam1_camera_center" link2="support2_link" reason="Never"/>
+    <disable_collisions link1="cam1_camera_center" link2="ur5e/base_link_inertia" reason="Never"/>
+    <disable_collisions link1="cam1_camera_center" link2="ur5e/shoulder_link" reason="Never"/>
+    <disable_collisions link1="cam1_camera_center" link2="wheel_1_link" reason="Never"/>
+    <disable_collisions link1="cam1_camera_center" link2="wheel_1_sup_link" reason="Never"/>
+    <disable_collisions link1="cam1_camera_center" link2="wheel_2_link" reason="Never"/>
+    <disable_collisions link1="cam1_camera_center" link2="wheel_2_sup_link" reason="Never"/>
+    <disable_collisions link1="cam1_camera_center" link2="wheel_3_link" reason="Never"/>
+    <disable_collisions link1="cam1_camera_center" link2="wheel_3_sup_link" reason="Never"/>
+    <disable_collisions link1="cam2_camera_center" link2="imu_link" reason="Never"/>
+    <disable_collisions link1="cam2_camera_center" link2="lidar1_link" reason="Never"/>
+    <disable_collisions link1="cam2_camera_center" link2="lidar2_link" reason="Never"/>
+    <disable_collisions link1="cam2_camera_center" link2="support1_link" reason="Never"/>
+    <disable_collisions link1="cam2_camera_center" link2="support2_link" reason="Never"/>
+    <disable_collisions link1="cam2_camera_center" link2="ur5e/base_link_inertia" reason="Never"/>
+    <disable_collisions link1="cam2_camera_center" link2="ur5e/shoulder_link" reason="Never"/>
+    <disable_collisions link1="cam2_camera_center" link2="wheel_1_link" reason="Never"/>
+    <disable_collisions link1="cam2_camera_center" link2="wheel_1_sup_link" reason="Never"/>
+    <disable_collisions link1="cam2_camera_center" link2="wheel_2_link" reason="Never"/>
+    <disable_collisions link1="cam2_camera_center" link2="wheel_2_sup_link" reason="Never"/>
+    <disable_collisions link1="cam2_camera_center" link2="wheel_3_link" reason="Never"/>
+    <disable_collisions link1="cam2_camera_center" link2="wheel_3_sup_link" reason="Never"/>
+    <disable_collisions link1="cam2_camera_center" link2="zed_eef_link" reason="Never"/>
     <disable_collisions link1="finger_1" link2="finger_2" reason="Never"/>
     <disable_collisions link1="finger_1" link2="gripper_base" reason="Adjacent"/>
-    <disable_collisions link1="finger_1" link2="wrist_1_link" reason="Never"/>
-    <disable_collisions link1="finger_1" link2="wrist_2_link" reason="Never"/>
-    <disable_collisions link1="finger_1" link2="wrist_3_link" reason="Never"/>
+    <disable_collisions link1="finger_1" link2="ur5e/wrist_1_link" reason="Never"/>
+    <disable_collisions link1="finger_1" link2="ur5e/wrist_2_link" reason="Never"/>
+    <disable_collisions link1="finger_1" link2="ur5e/wrist_3_link" reason="Never"/>
     <disable_collisions link1="finger_1" link2="zed_eef_link" reason="Never"/>
     <disable_collisions link1="finger_2" link2="gripper_base" reason="Adjacent"/>
-    <disable_collisions link1="finger_2" link2="wrist_1_link" reason="Never"/>
-    <disable_collisions link1="finger_2" link2="wrist_2_link" reason="Never"/>
-    <disable_collisions link1="finger_2" link2="wrist_3_link" reason="Never"/>
+    <disable_collisions link1="finger_2" link2="ur5e/wrist_1_link" reason="Never"/>
+    <disable_collisions link1="finger_2" link2="ur5e/wrist_2_link" reason="Never"/>
+    <disable_collisions link1="finger_2" link2="ur5e/wrist_3_link" reason="Never"/>
     <disable_collisions link1="finger_2" link2="zed_eef_link" reason="Never"/>
-    <disable_collisions link1="forearm_link" link2="upper_arm_link" reason="Adjacent"/>
-    <disable_collisions link1="forearm_link" link2="wrist_1_link" reason="Adjacent"/>
-    <disable_collisions link1="forearm_link" link2="wrist_2_link" reason="Never"/>
-    <disable_collisions link1="forearm_link" link2="zed_eef_link" reason="Never"/>
-    <disable_collisions link1="gripper_base" link2="wrist_1_link" reason="Never"/>
-    <disable_collisions link1="gripper_base" link2="wrist_2_link" reason="Never"/>
-    <disable_collisions link1="gripper_base" link2="wrist_3_link" reason="Adjacent"/>
+    <disable_collisions link1="gripper_base" link2="ur5e/wrist_1_link" reason="Never"/>
+    <disable_collisions link1="gripper_base" link2="ur5e/wrist_2_link" reason="Never"/>
+    <disable_collisions link1="gripper_base" link2="ur5e/wrist_3_link" reason="Adjacent"/>
     <disable_collisions link1="gripper_base" link2="zed_eef_link" reason="Adjacent"/>
-    <disable_collisions link1="shoulder_link" link2="upper_arm_link" reason="Adjacent"/>
-    <disable_collisions link1="shoulder_link" link2="zed_eef_link" reason="Never"/>
-    <disable_collisions link1="upper_arm_link" link2="zed_eef_link" reason="Never"/>
-    <disable_collisions link1="wrist_1_link" link2="wrist_2_link" reason="Adjacent"/>
-    <disable_collisions link1="wrist_1_link" link2="wrist_3_link" reason="Never"/>
-    <disable_collisions link1="wrist_1_link" link2="zed_eef_link" reason="Never"/>
-    <disable_collisions link1="wrist_2_link" link2="wrist_3_link" reason="Adjacent"/>
-    <disable_collisions link1="wrist_2_link" link2="zed_eef_link" reason="Never"/>
-    <disable_collisions link1="wrist_3_link" link2="zed_eef_link" reason="Adjacent"/>
+    <disable_collisions link1="imu_link" link2="lidar1_link" reason="Never"/>
+    <disable_collisions link1="imu_link" link2="lidar2_link" reason="Never"/>
+    <disable_collisions link1="imu_link" link2="support1_link" reason="Never"/>
+    <disable_collisions link1="imu_link" link2="support2_link" reason="Never"/>
+    <disable_collisions link1="imu_link" link2="ur5e/base_link_inertia" reason="Never"/>
+    <disable_collisions link1="imu_link" link2="ur5e/shoulder_link" reason="Never"/>
+    <disable_collisions link1="imu_link" link2="wheel_1_link" reason="Never"/>
+    <disable_collisions link1="imu_link" link2="wheel_1_sup_link" reason="Never"/>
+    <disable_collisions link1="imu_link" link2="wheel_2_link" reason="Never"/>
+    <disable_collisions link1="imu_link" link2="wheel_2_sup_link" reason="Never"/>
+    <disable_collisions link1="imu_link" link2="wheel_3_link" reason="Never"/>
+    <disable_collisions link1="imu_link" link2="wheel_3_sup_link" reason="Never"/>
+    <disable_collisions link1="lidar1_link" link2="lidar2_link" reason="Never"/>
+    <disable_collisions link1="lidar1_link" link2="support1_link" reason="Never"/>
+    <disable_collisions link1="lidar1_link" link2="support2_link" reason="Never"/>
+    <disable_collisions link1="lidar1_link" link2="ur5e/base_link_inertia" reason="Never"/>
+    <disable_collisions link1="lidar1_link" link2="ur5e/shoulder_link" reason="Never"/>
+    <disable_collisions link1="lidar1_link" link2="wheel_1_link" reason="Never"/>
+    <disable_collisions link1="lidar1_link" link2="wheel_1_sup_link" reason="Never"/>
+    <disable_collisions link1="lidar1_link" link2="wheel_2_link" reason="Never"/>
+    <disable_collisions link1="lidar1_link" link2="wheel_2_sup_link" reason="Never"/>
+    <disable_collisions link1="lidar1_link" link2="wheel_3_link" reason="Never"/>
+    <disable_collisions link1="lidar1_link" link2="wheel_3_sup_link" reason="Never"/>
+    <disable_collisions link1="lidar2_link" link2="support1_link" reason="Never"/>
+    <disable_collisions link1="lidar2_link" link2="support2_link" reason="Never"/>
+    <disable_collisions link1="lidar2_link" link2="ur5e/base_link_inertia" reason="Never"/>
+    <disable_collisions link1="lidar2_link" link2="ur5e/shoulder_link" reason="Never"/>
+    <disable_collisions link1="lidar2_link" link2="wheel_1_link" reason="Never"/>
+    <disable_collisions link1="lidar2_link" link2="wheel_1_sup_link" reason="Never"/>
+    <disable_collisions link1="lidar2_link" link2="wheel_2_link" reason="Never"/>
+    <disable_collisions link1="lidar2_link" link2="wheel_2_sup_link" reason="Never"/>
+    <disable_collisions link1="lidar2_link" link2="wheel_3_link" reason="Never"/>
+    <disable_collisions link1="lidar2_link" link2="wheel_3_sup_link" reason="Never"/>
+    <disable_collisions link1="support1_link" link2="support2_link" reason="Adjacent"/>
+    <disable_collisions link1="support1_link" link2="ur5e/base_link_inertia" reason="Never"/>
+    <disable_collisions link1="support1_link" link2="ur5e/shoulder_link" reason="Never"/>
+    <disable_collisions link1="support1_link" link2="wheel_1_link" reason="Never"/>
+    <disable_collisions link1="support1_link" link2="wheel_1_sup_link" reason="Never"/>
+    <disable_collisions link1="support1_link" link2="wheel_2_link" reason="Never"/>
+    <disable_collisions link1="support1_link" link2="wheel_2_sup_link" reason="Never"/>
+    <disable_collisions link1="support1_link" link2="wheel_3_link" reason="Never"/>
+    <disable_collisions link1="support1_link" link2="wheel_3_sup_link" reason="Never"/>
+    <disable_collisions link1="support2_link" link2="ur5e/base_link_inertia" reason="Never"/>
+    <disable_collisions link1="support2_link" link2="ur5e/forearm_link" reason="Default"/>
+    <disable_collisions link1="support2_link" link2="ur5e/shoulder_link" reason="Never"/>
+    <disable_collisions link1="support2_link" link2="ur5e/upper_arm_link" reason="Default"/>
+    <disable_collisions link1="support2_link" link2="wheel_1_link" reason="Never"/>
+    <disable_collisions link1="support2_link" link2="wheel_1_sup_link" reason="Never"/>
+    <disable_collisions link1="support2_link" link2="wheel_2_link" reason="Never"/>
+    <disable_collisions link1="support2_link" link2="wheel_2_sup_link" reason="Never"/>
+    <disable_collisions link1="support2_link" link2="wheel_3_link" reason="Never"/>
+    <disable_collisions link1="support2_link" link2="wheel_3_sup_link" reason="Never"/>
+    <disable_collisions link1="ur5e/base_link_inertia" link2="ur5e/shoulder_link" reason="Adjacent"/>
+    <disable_collisions link1="ur5e/base_link_inertia" link2="wheel_1_link" reason="Never"/>
+    <disable_collisions link1="ur5e/base_link_inertia" link2="wheel_1_sup_link" reason="Never"/>
+    <disable_collisions link1="ur5e/base_link_inertia" link2="wheel_2_link" reason="Never"/>
+    <disable_collisions link1="ur5e/base_link_inertia" link2="wheel_2_sup_link" reason="Never"/>
+    <disable_collisions link1="ur5e/base_link_inertia" link2="wheel_3_link" reason="Never"/>
+    <disable_collisions link1="ur5e/base_link_inertia" link2="wheel_3_sup_link" reason="Never"/>
+    <disable_collisions link1="ur5e/base_link_inertia" link2="zed_eef_link" reason="Never"/>
+    <disable_collisions link1="ur5e/forearm_link" link2="ur5e/upper_arm_link" reason="Adjacent"/>
+    <disable_collisions link1="ur5e/forearm_link" link2="ur5e/wrist_1_link" reason="Adjacent"/>
+    <disable_collisions link1="ur5e/forearm_link" link2="ur5e/wrist_2_link" reason="Never"/>
+    <disable_collisions link1="ur5e/forearm_link" link2="zed_eef_link" reason="Never"/>
+    <disable_collisions link1="ur5e/shoulder_link" link2="ur5e/upper_arm_link" reason="Adjacent"/>
+    <disable_collisions link1="ur5e/shoulder_link" link2="wheel_1_link" reason="Never"/>
+    <disable_collisions link1="ur5e/shoulder_link" link2="wheel_1_sup_link" reason="Never"/>
+    <disable_collisions link1="ur5e/shoulder_link" link2="wheel_2_link" reason="Never"/>
+    <disable_collisions link1="ur5e/shoulder_link" link2="wheel_2_sup_link" reason="Never"/>
+    <disable_collisions link1="ur5e/shoulder_link" link2="wheel_3_link" reason="Never"/>
+    <disable_collisions link1="ur5e/shoulder_link" link2="wheel_3_sup_link" reason="Never"/>
+    <disable_collisions link1="ur5e/shoulder_link" link2="zed_eef_link" reason="Never"/>
+    <disable_collisions link1="ur5e/upper_arm_link" link2="wheel_1_link" reason="Never"/>
+    <disable_collisions link1="ur5e/upper_arm_link" link2="wheel_1_sup_link" reason="Never"/>
+    <disable_collisions link1="ur5e/upper_arm_link" link2="wheel_2_link" reason="Never"/>
+    <disable_collisions link1="ur5e/upper_arm_link" link2="wheel_2_sup_link" reason="Never"/>
+    <disable_collisions link1="ur5e/upper_arm_link" link2="wheel_3_link" reason="Never"/>
+    <disable_collisions link1="ur5e/upper_arm_link" link2="wheel_3_sup_link" reason="Never"/>
+    <disable_collisions link1="ur5e/upper_arm_link" link2="zed_eef_link" reason="Never"/>
+    <disable_collisions link1="ur5e/wrist_1_link" link2="ur5e/wrist_2_link" reason="Adjacent"/>
+    <disable_collisions link1="ur5e/wrist_1_link" link2="ur5e/wrist_3_link" reason="Never"/>
+    <disable_collisions link1="ur5e/wrist_1_link" link2="zed_eef_link" reason="Never"/>
+    <disable_collisions link1="ur5e/wrist_2_link" link2="ur5e/wrist_3_link" reason="Adjacent"/>
+    <disable_collisions link1="ur5e/wrist_2_link" link2="zed_eef_link" reason="Never"/>
+    <disable_collisions link1="ur5e/wrist_3_link" link2="zed_eef_link" reason="Adjacent"/>
+    <disable_collisions link1="wheel_1_link" link2="wheel_1_sup_link" reason="Adjacent"/>
+    <disable_collisions link1="wheel_1_link" link2="wheel_2_link" reason="Never"/>
+    <disable_collisions link1="wheel_1_link" link2="wheel_2_sup_link" reason="Never"/>
+    <disable_collisions link1="wheel_1_link" link2="wheel_3_link" reason="Never"/>
+    <disable_collisions link1="wheel_1_link" link2="wheel_3_sup_link" reason="Never"/>
+    <disable_collisions link1="wheel_1_sup_link" link2="wheel_2_link" reason="Never"/>
+    <disable_collisions link1="wheel_1_sup_link" link2="wheel_2_sup_link" reason="Never"/>
+    <disable_collisions link1="wheel_1_sup_link" link2="wheel_3_link" reason="Never"/>
+    <disable_collisions link1="wheel_1_sup_link" link2="wheel_3_sup_link" reason="Never"/>
+    <disable_collisions link1="wheel_2_link" link2="wheel_2_sup_link" reason="Adjacent"/>
+    <disable_collisions link1="wheel_2_link" link2="wheel_3_link" reason="Never"/>
+    <disable_collisions link1="wheel_2_link" link2="wheel_3_sup_link" reason="Never"/>
+    <disable_collisions link1="wheel_2_sup_link" link2="wheel_3_link" reason="Never"/>
+    <disable_collisions link1="wheel_2_sup_link" link2="wheel_3_sup_link" reason="Never"/>
+    <disable_collisions link1="wheel_2_sup_link" link2="zed_eef_link" reason="Never"/>
+    <disable_collisions link1="wheel_3_link" link2="wheel_3_sup_link" reason="Adjacent"/>
+    <disable_collisions link1="wheel_3_sup_link" link2="zed_eef_link" reason="Never"/>
   </xacro:macro>
 </robot>

File: robot_ws_ros2/src/call_m_supervisor/urdf/sim.urdf.xacro (robot description, xacro)
@@ -1,4 +1,11 @@
 <?xml version="1.0"?>
 <robot xmlns:xacro="http://wiki.ros.org/xacro" name="call_m_arm">
+	<link name="world">
+	</link>
+	<joint name="world-base_link" type="fixed">
+		<parent link="world"/>
+		<child link="base_link"/>
+		<origin xyz="0.0 -1.0 0.2" rpy="0.0 0.0 0.0"/>
+	</joint>
   	<!-- Define robot constants -->
 	<!-- If changed, check also 'simu_bot_driver.cpp' for publish_command() -->
@@ -247,5 +254,5 @@
    <xacro:arg name="ur_type" default="ur5e"/>
    <!-- parameters -->
-   <xacro:arg name="tf_prefix" default="/ur5e/" />
+   <xacro:arg name="tf_prefix" default="ur5e/" />
    <xacro:arg name="joint_limit_params" default="$(find ur_description)/config/$(arg ur_type)/joint_limits.yaml"/>
    <xacro:arg name="kinematics_params" default="$(find ur_description)/config/$(arg ur_type)/default_kinematics.yaml"/>
